Commit message: Modifications: UR3 Gz package.

File: ur3cranfield_gazebo/urdf/ur3_common.xacro (robot description, xacro)
@@ -17,9 +17,10 @@
 #                                                                                       #
 #  IFRA Group - Cranfield University                                                    #
-#  AUTHORS: Mikel Bueno Viso - Mikel.Bueno-Viso@cranfield.ac.uk                         #
-#           Dr. Seemal Asif  - s.asif@cranfield.ac.uk                                   #
-#           Prof. Phil Webb  - p.f.webb@cranfield.ac.uk                                 #
+#  AUTHORS: Mikel Bueno Viso - Mikel.Bueno-Viso@cranfield.ac.uk     (ROS 2 Packages)    #
+#           James Fowler     - j.fowler@cranfield.ac.uk             (UR3 Cell Design)   #
+#           Daniel Oakley    - daniel.oakley@cranfield.ac.uk        (UR3 Cell Design)   #
+#           Jamie Rice       - jamie.rice@cranfield.ac.uk           (UR3 Cell Design)   #
 #                                                                                       #
-#  Date: May, 2023.                                                                     #
+#  Date: April, 2024.                                                                   #
 #                                                                                       #
 # ===================================== COPYRIGHT ===================================== #
@@ -53,4 +54,5 @@
 # You can cite our work with the following statement:
 # IFRA-Cranfield (2023) ROS 2 Sim-to-Real Robot Control. URL: https://github.com/IFRA-Cranfield/ros2_SimRealRobotControl.
+# IFRA-Cranfield (2024) UR3 Cranfield Robotics Cell. URL: https://github.com/IFRA-Cranfield/ur3_CranfieldRobotics.
 -->
 <robot xmlns:xacro="http://wiki.ros.org/xacro">

File: ur3cranfield_gazebo/urdf/ur3_macro.urdf.xacro (robot description, xacro)
@@ -324,11 +324,20 @@
       </visual>
     </link>
-    <joint name="BASE_TF_joint" type="prismatic" >
-      <parent link="base_link" />
-      <child link="BASE_TF" />
-      <limit effort="10000" lower="0.0" upper="0.0" velocity="0.0"/>
-      <axis xyz="1 0 0" />
-      <origin xyz="0.0 0.0 0.0" rpy="0 0 0"/>
-    </joint>
+    <xacro:unless value="${bringup}">
+      <joint name="BASE_TF_joint" type="prismatic" >
+        <parent link="base_link" />
+        <child link="BASE_TF" />
+        <limit effort="10000" lower="0.0" upper="0.0" velocity="0.0"/>
+        <axis xyz="1 0 0" />
+        <origin xyz="0.0 0.0 0.0" rpy="0 0 0"/>
+      </joint>
+    </xacro:unless>
+    <xacro:if value="${bringup}">
+      <joint name="BASE_TF_joint" type="fixed" >
+        <parent link="base_link" />
+        <child link="BASE_TF" />
+        <origin xyz="0.0 0.0 0.0" rpy="0 0 0"/>
+      </joint>
+    </xacro:if>
     <!-- EXTRA LINK + JOINT for the TCP to appear in Gazebo and to be able to calculate TRANSFORMS: -->
     <link name="TCP">
@@ -344,13 +353,20 @@
       </visual>
     </link>
-    <joint name="TCP_joint" type="prismatic" >
-      <parent link="wrist_3_link" />
-      <child link="TCP" />
-      <limit effort="10000" lower="0.0" upper="0.0" velocity="0.0"/>
-      <axis xyz="1 0 0" />
-      <origin xyz="0.0 0.0 0.0" rpy="0 0 0"/>
-    </joint>
-    <!-- =================================== -->
-    <!-- ========== END-EFFECTORS ========== -->
+    <xacro:unless value="${bringup}">
+      <joint name="TCP_joint" type="prismatic" >
+        <parent link="wrist_3_link" />
+        <child link="TCP" />
+        <limit effort="10000" lower="0.0" upper="0.0" velocity="0.0"/>
+        <axis xyz="1 0 0" />
+        <origin xyz="0.0 0.0 0.0" rpy="0 0 0"/>
+      </joint>
+    </xacro:unless>
+    <xacro:if value="${bringup}">
+      <joint name="TCP_joint" type="fixed" >
+        <parent link="wrist_3_link" />
+        <child link="TCP" />
+        <origin xyz="0.0 0.0 0.0" rpy="0 0 0"/>
+      </joint>
+    </xacro:if>
     <!-- === ROBOTIQ 2f-85 GRIPPER === -->
     <!-- NOTE: JOINT LIMITS have been slightly augmentated from 0.0 to +-0.05 to avoid errors in MoveIt!2 execution. -->
@@ -642,13 +658,27 @@
       </visual>
     </link>
-    <joint name="EE_robotiq_2f85_joint" type="prismatic" >
-      <parent link="robotiq_85_base_link" />
-      <child link="EE_robotiq_2f85" />
-      <limit effort="10000" lower="0.0" upper="0.0" velocity="0.0"/>
-      <axis xyz="1 0 0" />
-      <origin xyz="0.128 0.0 0.0" rpy="0 0 0"/>
-    </joint>
+    <xacro:unless value="${bringup}">
+      <joint name="EE_robotiq_2f85_joint" type="prismatic" >
+        <parent link="robotiq_85_base_link" />
+        <child link="EE_robotiq_2f85" />
+        <limit effort="10000" lower="0.0" upper="0.0" velocity="0.0"/>
+        <axis xyz="1 0 0" />
+        <origin xyz="0.128 0.0 0.0" rpy="0 0 0"/>
+      </joint>
+      <!-- LOAD LinkPose Gazebo (ROS2) PLUGIN: -->
+      <gazebo>
+        <plugin name="ros2_linkpose_plugin" filename="libros2_linkpose_plugin.so" >
+          <link>EE_robotiq_2f85</link>
+        </plugin>
+      </gazebo>
+    </xacro:unless>
+    <xacro:if value="${bringup}">
+      <joint name="EE_robotiq_2f85_joint" type="fixed" >
+        <parent link="robotiq_85_base_link" />
+        <child link="EE_robotiq_2f85" />
+        <origin xyz="0.128 0.0 0.0" rpy="0 0 0"/>
+      </joint>
+    </xacro:if>
     <!-- === ROBOTIQ 2f-85 GRIPPER === -->
-    <!-- ========== END-EFFECTORS ========== -->
   </xacro:macro>
 </robot>

File: ur3cranfield_gazebo/urdf/ur3_ros2control.xacro (robot description, xacro)
@@ -336,4 +336,24 @@
       </joint>
       <!-- === ROBOTIQ 2f-85 GRIPPER === -->
+      <xacro:unless value="${bringup}">
+        <joint name="BASE_TF_joint">
+          <command_interface name="position"/>
+          <command_interface name="velocity"/>
+          <state_interface name="position"/>
+          <state_interface name="velocity"/>
+        </joint>
+        <joint name="TCP_joint">
+          <command_interface name="position"/>
+          <command_interface name="velocity"/>
+          <state_interface name="position"/>
+          <state_interface name="velocity"/>
+        </joint>
+        <joint name="EE_robotiq_2f85_joint">
+          <command_interface name="position"/>
+          <command_interface name="velocity"/>
+          <state_interface name="position"/>
+          <state_interface name="velocity"/>
+        </joint>
+      </xacro:unless>
     </ros2_control>
     <xacro:unless value="${bringup}">

Commit message: Fix params for UR3 - ROS 2 connection (working, but with execution errors).

File: ur3cranfield_gazebo/urdf/ur3_common.xacro (robot description, xacro)
@@ -190,5 +190,5 @@
     <xacro:property name="wrist_3_visual_offset" value="-0.082" scope="parent"/>
     <!--KINEMATICS HASH-->
-    <xacro:property name="kinematics_hash" value="calib_9122066269688285636" scope="parent"/>
+    <xacro:property name="kinematics_hash" value="calib_604802427893924187" scope="parent"/>
   </xacro:macro>
 </robot>

File: ur3cranfield_gazebo/urdf/ur3_ros2control.xacro (robot description, xacro)
@@ -80,5 +80,5 @@
   <xacro:arg name="use_tool_communication" default="false"/>
   <xacro:property name="use_tool_communication" value="$(arg use_tool_communication)"/>
-  <xacro:arg name="hash_kinematics" default="calib_9122066269688285636"/>
+  <xacro:arg name="hash_kinematics" default="calib_604802427893924187"/>
   <xacro:property name="hash_kinematics" value="$(arg hash_kinematics)"/>
   <xacro:arg name="tool_voltage" default="24"/>
