Commit message: Update: UR3 IA Lab stand (w/ box).

File: ur3cranfield_gazebo/urdf/ur3.urdf.xacro (robot description, xacro)
@@ -84,5 +84,5 @@
       <origin xyz="0.0 0.0 0.0" rpy="0 0 0" />
       <geometry>
-        <mesh filename="file://$(find ur3cranfield_gazebo)/meshes/ur3stand/ur3stand_NoBox.dae" scale="1 1 1" />
+        <mesh filename="file://$(find ur3cranfield_gazebo)/meshes/ur3stand/ur3stand.dae" scale="1 1 1" />
       </geometry>
     </visual>
@@ -90,5 +90,5 @@
       <origin xyz="0.0 0.0 0.0" rpy="0 0 0" />
       <geometry>
-        <mesh filename="file://$(find ur3cranfield_gazebo)/meshes/ur3stand/ur3stand_NoBox.dae" scale="1 1 1" />
+        <mesh filename="file://$(find ur3cranfield_gazebo)/meshes/ur3stand/ur3stand.dae" scale="1 1 1" />
       </geometry>
     </collision>

File: ur3cranfield_gazebo/urdf/ur3_ros2control.xacro (robot description, xacro)
@@ -224,5 +224,5 @@
         </command_interface>
         <state_interface name="position">
-          <param name="initial_value">0.0</param>
+          <param name="initial_value">${pi/2}</param>
         </state_interface>
         <state_interface name="velocity"/>

Commit message: Adapt for proper bringup and connection to ur3 (not working).

File: ur3cranfield_gazebo/urdf/ur3.urdf.xacro (robot description, xacro)
@@ -106,5 +106,5 @@
     <parent link="ur3_stand" />
     <child link = "base_link" />
-    <origin xyz="0.0 0.0 0.85" rpy="0.0 0.0 0.0" />
+    <origin xyz="0.0 0.0 0.85" rpy="0.0 0.0 ${pi}" />
   </joint>
 </robot>

File: ur3cranfield_gazebo/urdf/ur3_ros2control.xacro (robot description, xacro)
@@ -209,5 +209,5 @@
         </command_interface>
         <state_interface name="position">
-          <param name="initial_value">0.0</param>
+          <param name="initial_value">${-pi/2}</param>
         </state_interface>
         <state_interface name="velocity"/>
@@ -224,5 +224,5 @@
         </command_interface>
         <state_interface name="position">
-          <param name="initial_value">${pi/2}</param>
+          <param name="initial_value">0.0</param>
         </state_interface>
         <state_interface name="velocity"/>

Commit message: Adapt ur3cranfield ROS 2 packages for bringup connection (works!).

File: ur3cranfield_gazebo/urdf/ur3.urdf.xacro (robot description, xacro)
@@ -68,4 +68,6 @@
   <xacro:arg name="output_recipe_filename" default="none"/>
   <xacro:property name="output_recipe_filename" value="$(arg output_recipe_filename)"/>
+  <xacro:arg name="tf_prefix" default=""/>
+  <xacro:property name="tf_prefix" value="$(arg tf_prefix)"/>
   <!-- Include XACRO-MACRO file of the UR3: -->
   <xacro:include filename="$(find ur3cranfield_gazebo)/urdf/ur3_macro.urdf.xacro"/>
@@ -76,9 +78,10 @@
     input_recipe_filename="${input_recipe_filename}"
     output_recipe_filename="${output_recipe_filename}"
+    tf_prefix="${tf_prefix}"
     />
   <!-- World link -->
   <link name="world"/>
   <!-- === Cranfield Robotics UR3 Cell === -->
-  <link name='ur3_stand'>
+  <link name='${tf_prefix}ur3_stand'>
     <visual>
       <origin xyz="0.0 0.0 0.0" rpy="0 0 0" />
@@ -98,12 +101,12 @@
     </inertial>
   </link>
-  <joint name="world_joint" type="fixed">
+  <joint name="${tf_prefix}world_joint" type="fixed">
       <parent link="world" />
-      <child link = "ur3_stand" />
+      <child link = "${tf_prefix}ur3_stand" />
       <origin xyz="0.0 0.0 0.0" rpy="0.0 0.0 0.0" />
     </joint>
-  <joint name="ur_joint" type="fixed">
-    <parent link="ur3_stand" />
-    <child link = "base_link" />
+  <joint name="${tf_prefix}ur_joint" type="fixed">
+    <parent link="${tf_prefix}ur3_stand" />
+    <child link = "${tf_prefix}base_link" />
     <origin xyz="0.0 0.0 0.85" rpy="0.0 0.0 ${pi}" />
   </joint>

File: ur3cranfield_gazebo/urdf/ur3_macro.urdf.xacro (robot description, xacro)
@@ -60,5 +60,5 @@
   <xacro:include filename="$(find ur3cranfield_gazebo)/urdf/ur3_common.xacro" />
   <!-- XACRO-MACRO of UR3: -->
-  <xacro:macro name="ur3" params="bringup robot_ip script_filename input_recipe_filename output_recipe_filename">
+  <xacro:macro name="ur3" params="bringup robot_ip script_filename input_recipe_filename output_recipe_filename tf_prefix">
     <!-- LOAD UR3-Common: -->
     <xacro:ur3_common/>
@@ -75,9 +75,10 @@
       script_filename="${script_filename}"
       input_recipe_filename="${input_recipe_filename}"
-      output_recipe_filename="${output_recipe_filename}"/>
+      output_recipe_filename="${output_recipe_filename}"
+      tf_prefix="${tf_prefix}"/>
     <!-- ***** UR3 ROBOT .urdf SERIAL CHAIN ***** -->
     <!-- Links: -->
-    <link name="base_link"/>
-    <link name="base_link_inertia">
+    <link name="${tf_prefix}base_link"/>
+    <link name="${tf_prefix}base_link_inertia">
       <visual>
         <origin xyz="0 0 0" rpy="0 0 ${pi}"/>
@@ -99,5 +100,5 @@
       </xacro:cylinder_inertial>
     </link>
-    <link name="shoulder_link">
+    <link name="${tf_prefix}shoulder_link">
       <visual>
         <origin xyz="0 0 0" rpy="0 0 ${pi}"/>
@@ -119,5 +120,5 @@
       </xacro:cylinder_inertial>
     </link>
-    <link name="upper_arm_link">
+    <link name="${tf_prefix}upper_arm_link">
       <visual>
         <origin xyz="0 0 ${shoulder_offset}" rpy="${pi/2} 0 ${-pi/2}"/>
@@ -139,5 +140,5 @@
       </xacro:cylinder_inertial>
     </link>
-    <link name="forearm_link">
+    <link name="${tf_prefix}forearm_link">
       <visual>
         <origin xyz="0 0 ${elbow_offset}" rpy="${pi/2} 0 ${-pi/2}"/>
@@ -159,5 +160,5 @@
       </xacro:cylinder_inertial>
     </link>
-    <link name="wrist_1_link">
+    <link name="${tf_prefix}wrist_1_link">
       <visual>
         <origin xyz="0 0 ${wrist_1_visual_offset}" rpy="${pi/2} 0 0"/>
@@ -179,5 +180,5 @@
       </xacro:cylinder_inertial>
     </link>
-    <link name="wrist_2_link">
+    <link name="${tf_prefix}wrist_2_link">
       <visual>
         <origin xyz="0 0 ${wrist_2_visual_offset}" rpy="0 0 0"/>
@@ -199,5 +200,5 @@
       </xacro:cylinder_inertial>
     </link>
-    <link name="wrist_3_link">
+    <link name="${tf_prefix}wrist_3_link">
       <visual>
         <origin xyz="0 0 ${wrist_3_visual_offset}" rpy="${pi/2} 0 0"/>
@@ -220,7 +221,7 @@
     </link>
     <!-- Joints: -->
-    <joint name="base_link-base_link_inertia" type="fixed">
-      <parent link="base_link" />
-      <child link="base_link_inertia" />
+    <joint name="${tf_prefix}base_link-base_link_inertia" type="fixed">
+      <parent link="${tf_prefix}base_link" />
+      <child link="${tf_prefix}base_link_inertia" />
       <!-- 'base_link' is REP-103 aligned (so X+ forward), while the internal
            frames of the robot/controller have X+ pointing backwards.
@@ -230,7 +231,7 @@
       <origin xyz="0 0 0" rpy="0 0 ${pi}" />
     </joint>
-    <joint name="shoulder_pan_joint" type="revolute">
-      <parent link="base_link_inertia" />
-      <child link="shoulder_link" />
+    <joint name="${tf_prefix}shoulder_pan_joint" type="revolute">
+      <parent link="${tf_prefix}base_link_inertia" />
+      <child link="${tf_prefix}shoulder_link" />
       <origin xyz="${shoulder_x} ${shoulder_y} ${shoulder_z}" rpy="${shoulder_roll} ${shoulder_pitch} ${shoulder_yaw}" />
       <axis xyz="0 0 1" />
@@ -239,7 +240,7 @@
       <dynamics damping="1.0" friction="100.0"/>
     </joint>
-    <joint name="shoulder_lift_joint" type="revolute">
-      <parent link="shoulder_link" />
-      <child link="upper_arm_link" />
+    <joint name="${tf_prefix}shoulder_lift_joint" type="revolute">
+      <parent link="${tf_prefix}shoulder_link" />
+      <child link="${tf_prefix}upper_arm_link" />
       <origin xyz="${upper_arm_x} ${upper_arm_y} ${upper_arm_z}" rpy="${upper_arm_roll} ${upper_arm_pitch} ${upper_arm_yaw}" />
       <axis xyz="0 0 1" />
@@ -248,7 +249,7 @@
       <dynamics damping="1.0" friction="100.0"/>
     </joint>
-    <joint name="elbow_joint" type="revolute">
-      <parent link="upper_arm_link" />
-      <child link="forearm_link" />
+    <joint name="${tf_prefix}elbow_joint" type="revolute">
+      <parent link="${tf_prefix}upper_arm_link" />
+      <child link="${tf_prefix}forearm_link" />
       <origin xyz="${forearm_x} ${forearm_y} ${forearm_z}" rpy="${forearm_roll} ${forearm_pitch} ${forearm_yaw}" />
       <axis xyz="0 0 1" />
@@ -257,7 +258,7 @@
       <dynamics damping="1.0" friction="100.0"/>
     </joint>
-    <joint name="wrist_1_joint" type="revolute">
-      <parent link="forearm_link" />
-      <child link="wrist_1_link" />
+    <joint name="${tf_prefix}wrist_1_joint" type="revolute">
+      <parent link="${tf_prefix}forearm_link" />
+      <child link="${tf_prefix}wrist_1_link" />
       <origin xyz="${wrist_1_x} ${wrist_1_y} ${wrist_1_z}" rpy="${wrist_1_roll} ${wrist_1_pitch} ${wrist_1_yaw}" />
       <axis xyz="0 0 1" />
@@ -266,7 +267,7 @@
       <dynamics damping="1.0" friction="10.0"/>
     </joint>
-    <joint name="wrist_2_joint" type="revolute">
-      <parent link="wrist_1_link" />
-      <child link="wrist_2_link" />
+    <joint name="${tf_prefix}wrist_2_joint" type="revolute">
+      <parent link="${tf_prefix}wrist_1_link" />
+      <child link="${tf_prefix}wrist_2_link" />
       <origin xyz="${wrist_2_x} ${wrist_2_y} ${wrist_2_z}" rpy="${wrist_2_roll} ${wrist_2_pitch} ${wrist_2_yaw}" />
       <axis xyz="0 0 1" />
@@ -275,7 +276,7 @@
       <dynamics damping="1.0" friction="10.0"/>
     </joint>
-    <joint name="wrist_3_joint" type="revolute">
-      <parent link="wrist_2_link" />
-      <child link="wrist_3_link" />
+    <joint name="${tf_prefix}wrist_3_joint" type="revolute">
+      <parent link="${tf_prefix}wrist_2_link" />
+      <child link="${tf_prefix}wrist_3_link" />
       <origin xyz="${wrist_3_x} ${wrist_3_y} ${wrist_3_z}" rpy="${wrist_3_roll} ${wrist_3_pitch} ${wrist_3_yaw}" />
       <axis xyz="0 0 1" />
@@ -285,6 +286,6 @@
     </joint>
     <!-- ROS-Industrial 'base' frame - base_link to UR 'Base' Coordinates transform -->
-    <link name="base"/>
-    <joint name="base_link-base_fixed_joint" type="fixed">
+    <link name="${tf_prefix}base"/>
+    <joint name="${tf_prefix}base_link-base_fixed_joint" type="fixed">
       <!-- Note the rotation over Z of pi radians - as base_link is REP-103
            aligned (i.e., has X+ forward, Y+ left and Z+ up), this is needed
@@ -293,24 +294,24 @@
       -->
       <origin xyz="0 0 0" rpy="0 0 ${pi}"/>
-      <parent link="base_link"/>
-      <child link="base"/>
+      <parent link="${tf_prefix}base_link"/>
+      <child link="${tf_prefix}base"/>
     </joint>
     <!-- ROS-Industrial 'flange' frame - attachment point for EEF models -->
-    <link name="flange" />
-    <joint name="wrist_3-flange" type="fixed">
-      <parent link="wrist_3_link" />
-      <child link="flange" />
+    <link name="${tf_prefix}flange" />
+    <joint name="${tf_prefix}wrist_3-flange" type="fixed">
+      <parent link="${tf_prefix}wrist_3_link" />
+      <child link="${tf_prefix}flange" />
       <origin xyz="0 0 0" rpy="0 ${-pi/2.0} ${-pi/2.0}" />
     </joint>
     <!-- ROS-Industrial 'tool0' frame - all-zeros tool frame -->
-    <link name="tool0"/>
-    <joint name="flange-tool0" type="fixed">
+    <link name="${tf_prefix}tool0"/>
+    <joint name="${tf_prefix}flange-tool0" type="fixed">
       <!-- default toolframe - X+ left, Y+ up, Z+ front -->
       <origin xyz="0 0 0" rpy="${pi/2.0} 0 ${pi/2.0}"/>
-      <parent link="flange"/>
-      <child link="tool0"/>
+      <parent link="${tf_prefix}flange"/>
+      <child link="${tf_prefix}tool0"/>
     </joint>
     <!-- EXTRA LINK + JOINT for the base_link to appear in Gazebo and to be able to calculate TRANSFORMS: -->
-    <link name="BASE_TF">
+    <link name="${tf_prefix}BASE_TF">
       <inertial>
         <origin xyz="0 0 0" rpy="0 0 0" />
@@ -325,7 +326,7 @@
     </link>
     <xacro:unless value="${bringup}">
-      <joint name="BASE_TF_joint" type="prismatic" >
-        <parent link="base_link" />
-        <child link="BASE_TF" />
+      <joint name="${tf_prefix}BASE_TF_joint" type="prismatic" >
+        <parent link="${tf_prefix}base_link" />
+        <child link="${tf_prefix}BASE_TF" />
         <limit effort="10000" lower="0.0" upper="0.0" velocity="0.0"/>
         <axis xyz="1 0 0" />
@@ -334,12 +335,12 @@
     </xacro:unless>
     <xacro:if value="${bringup}">
-      <joint name="BASE_TF_joint" type="fixed" >
-        <parent link="base_link" />
-        <child link="BASE_TF" />
+      <joint name="${tf_prefix}BASE_TF_joint" type="fixed" >
+        <parent link="${tf_prefix}base_link" />
+        <child link="${tf_prefix}BASE_TF" />
         <origin xyz="0.0 0.0 0.0" rpy="0 0 0"/>
       </joint>
     </xacro:if>
     <!-- EXTRA LINK + JOINT for the TCP to appear in Gazebo and to be able to calculate TRANSFORMS: -->
-    <link name="TCP">
+    <link name="${tf_prefix}TCP">
       <inertial>
         <origin xyz="0 0 0" rpy="0 0 0" />
@@ -354,7 +355,7 @@
     </link>
     <xacro:unless value="${bringup}">
-      <joint name="TCP_joint" type="prismatic" >
-        <parent link="wrist_3_link" />
-        <child link="TCP" />
+      <joint name="${tf_prefix}TCP_joint" type="prismatic" >
+        <parent link="${tf_prefix}wrist_3_link" />
+        <child link="${tf_prefix}TCP" />
         <limit effort="10000" lower="0.0" upper="0.0" velocity="0.0"/>
         <axis xyz="1 0 0" />
@@ -363,7 +364,7 @@
     </xacro:unless>
     <xacro:if value="${bringup}">
-      <joint name="TCP_joint" type="fixed" >
-        <parent link="wrist_3_link" />
-        <child link="TCP" />
+      <joint name="${tf_prefix}TCP_joint" type="fixed" >
+        <parent link="${tf_prefix}wrist_3_link" />
+        <child link="${tf_prefix}TCP" />
         <origin xyz="0.0 0.0 0.0" rpy="0 0 0"/>
       </joint>
