Commit message: Update stand, add aruco tags and Gz cameras.

File: ur3cranfield_gazebo/urdf/ur3.urdf.xacro (robot description, xacro)
@@ -87,5 +87,5 @@
       <origin xyz="0.0 0.0 0.0" rpy="0 0 0" />
       <geometry>
-        <mesh filename="file://$(find ur3cranfield_gazebo)/meshes/ur3stand/ur3stand.dae" scale="1 1 1" />
+        <mesh filename="file://$(find ur3cranfield_gazebo)/meshes/ur3stand/ur3stand_complete.dae" scale="1 1 1" />
       </geometry>
     </visual>
@@ -93,5 +93,5 @@
       <origin xyz="0.0 0.0 0.0" rpy="0 0 0" />
       <geometry>
-        <mesh filename="file://$(find ur3cranfield_gazebo)/meshes/ur3stand/ur3stand.dae" scale="1 1 1" />
+        <mesh filename="file://$(find ur3cranfield_gazebo)/meshes/ur3stand/ur3stand_complete.dae" scale="1 1 1" />
       </geometry>
     </collision>
@@ -111,3 +111,214 @@
     <origin xyz="0.0 0.0 0.85" rpy="0.0 0.0 ${pi}" />
   </joint>
+  <!-- ARUCO TAGS -->
+  <xacro:unless value="${bringup}">
+    <link name="aruco100">
+      <visual>
+        <origin xyz="0.0 0.0 0.0" rpy="0 0 0" />
+        <geometry>
+          <mesh filename="file://$(find ur3cranfield_gazebo)/meshes/aruco/aruco100.dae" scale="1 1 1" />
+        </geometry>
+      </visual>
+      <collision>
+        <origin xyz="0.0 0.0 0.0" rpy="0 0 0" />
+        <geometry>
+          <mesh filename="file://$(find ur3cranfield_gazebo)/meshes/aruco/aruco100.dae" scale="1 1 1" />
+        </geometry>
+      </collision>
+      <inertial>
+        <mass value="10.0"/>
+        <inertia ixx="0.0002" ixy="0.0002" ixz="0.0002" iyy="0.0" iyz="0.0" izz="0.0" />
+      </inertial>
+    </link>
+    <joint name="stand-aruco100-fixed" type="fixed">
+      <parent link="${tf_prefix}ur3_stand"/>
+      <child link="aruco100"/>
+      <origin xyz="-0.26 0.365 0.845" rpy="0.0 0.0 3.1416" />
+    </joint>
+    <link name="aruco101">
+      <visual>
+        <origin xyz="0.0 0.0 0.0" rpy="0 0 0" />
+        <geometry>
+          <mesh filename="file://$(find ur3cranfield_gazebo)/meshes/aruco/aruco101.dae" scale="1 1 1" />
+        </geometry>
+      </visual>
+      <collision>
+        <origin xyz="0.0 0.0 0.0" rpy="0 0 0" />
+        <geometry>
+          <mesh filename="file://$(find ur3cranfield_gazebo)/meshes/aruco/aruco101.dae" scale="1 1 1" />
+        </geometry>
+      </collision>
+      <inertial>
+        <mass value="10.0"/>
+        <inertia ixx="0.0002" ixy="0.0002" ixz="0.0002" iyy="0.0" iyz="0.0" izz="0.0" />
+      </inertial>
+    </link>
+    <joint name="stand-aruco101-fixed" type="fixed">
+      <parent link="${tf_prefix}ur3_stand"/>
+      <child link="aruco101"/>
+      <origin xyz="0.26 0.365 0.845" rpy="0.0 0.0 1.5708" />
+    </joint>
+    <link name="aruco102">
+      <visual>
+        <origin xyz="0.0 0.0 0.0" rpy="0 0 0" />
+        <geometry>
+          <mesh filename="file://$(find ur3cranfield_gazebo)/meshes/aruco/aruco102.dae" scale="1 1 1" />
+        </geometry>
+      </visual>
+      <collision>
+        <origin xyz="0.0 0.0 0.0" rpy="0 0 0" />
+        <geometry>
+          <mesh filename="file://$(find ur3cranfield_gazebo)/meshes/aruco/aruco102.dae" scale="1 1 1" />
+        </geometry>
+      </collision>
+      <inertial>
+        <mass value="10.0"/>
+        <inertia ixx="0.0002" ixy="0.0002" ixz="0.0002" iyy="0.0" iyz="0.0" izz="0.0" />
+      </inertial>
+    </link>
+    <joint name="stand-aruco102-fixed" type="fixed">
+      <parent link="${tf_prefix}ur3_stand"/>
+      <child link="aruco102"/>
+      <origin xyz="-0.26 0.115 0.845" rpy="0.0 0.0 -1.5708" />
+    </joint>
+    <link name="aruco103">
+      <visual>
+        <origin xyz="0.0 0.0 0.0" rpy="0 0 0" />
+        <geometry>
+          <mesh filename="file://$(find ur3cranfield_gazebo)/meshes/aruco/aruco103.dae" scale="1 1 1" />
+        </geometry>
+      </visual>
+      <collision>
+        <origin xyz="0.0 0.0 0.0" rpy="0 0 0" />
+        <geometry>
+          <mesh filename="file://$(find ur3cranfield_gazebo)/meshes/aruco/aruco103.dae" scale="1 1 1" />
+        </geometry>
+      </collision>
+      <inertial>
+        <mass value="10.0"/>
+        <inertia ixx="0.0002" ixy="0.0002" ixz="0.0002" iyy="0.0" iyz="0.0" izz="0.0" />
+      </inertial>
+    </link>
+    <joint name="stand-aruco103-fixed" type="fixed">
+      <parent link="${tf_prefix}ur3_stand"/>
+      <child link="aruco103"/>
+      <origin xyz="0.26 0.115 0.845" rpy="0.0 0.0 0.0" />
+    </joint>
+  </xacro:unless>
+  <!-- CAMERA -->
+  <xacro:unless value="${bringup}">
+    <link name="camera_link">
+      <collision>
+        <origin xyz="0 0 0" rpy="0 0 0"/>
+        <geometry>
+          <box size="0.05 0.05 0.05"/>
+        </geometry>
+      </collision>
+      <visual>
+        <origin xyz="0 0 0" rpy="0 0 0"/>
+        <geometry>
+          <box size="0.05 0.05 0.05"/>
+        </geometry>
+      </visual>
+      <inertial>
+        <mass value="1.0" />
+        <origin xyz="0 0 0" rpy="0 0 0"/>
+        <inertia ixx="0.0" ixy="0.0" ixz="0.0" iyy="0.0" iyz="0.0" izz="0.0" />
+      </inertial>
+    </link>
+    <joint name="camera_joint" type="fixed">
+      <origin xyz="0.0 0.32 2.09" rpy="0.0 1.5708 1.5708"/>
+      <parent link="world"/>
+      <child link="camera_link"/>
+    </joint>
+    <gazebo reference="camera_link">
+      <sensor name="camera" type="camera">
+        <update_rate>30</update_rate>
+        <camera name="head">
+          <horizontal_fov>1.22</horizontal_fov>
+          <image>
+            <width>1920</width>
+            <height>1080</height>
+            <format>R8G8B8</format>
+          </image>
+          <clip>
+            <near>0.02</near>
+            <far>300</far>
+          </clip>
+          <noise>
+            <type>gaussian</type>
+            <mean>0.0</mean>
+            <stddev>0.007</stddev>
+          </noise>
+        </camera>
+        <plugin filename="libgazebo_ros_camera.so" name="camera_controller">
+          <robotNamespace/>
+          <alwaysOn>true</alwaysOn>
+          <updateRate>0.0</updateRate>
+          <cameraName>camera</cameraName>
+          <imageTopicName>image_raw</imageTopicName>
+          <cameraInfoTopicName>camera_info</cameraInfoTopicName>
+          <frameName>camera</frameName>
+          <hackBaseline>0.07</hackBaseline>
+        </plugin>
+      </sensor>
+    </gazebo>
+    <!-- CAMERA for R3M-HMI -->
+    <link name="HMI_camera_link">
+      <collision>
+        <origin xyz="0 0 0" rpy="0 0 0"/>
+        <geometry>
+          <box size="0.05 0.05 0.05"/>
+        </geometry>
+      </collision>
+      <visual>
+        <origin xyz="0 0 0" rpy="0 0 0"/>
+        <geometry>
+          <box size="0.05 0.05 0.05"/>
+        </geometry>
+      </visual>
+      <inertial>
+        <mass value="1.0" />
+        <origin xyz="0 0 0" rpy="0 0 0"/>
+        <inertia ixx="0.0" ixy="0.0" ixz="0.0" iyy="0.0" iyz="0.0" izz="0.0" />
+      </inertial>
+    </link>
+    <joint name="HMI_camera_joint" type="fixed">
+      <origin xyz="2.0 1.5 2.0" rpy="0 0.35 -2.6"/>
+      <parent link="world"/>
+      <child link="HMI_camera_link"/>
+    </joint>
+    <gazebo reference="HMI_camera_link">
+      <sensor name="HMI_camera" type="camera">
+        <update_rate>30</update_rate>
+        <camera name="head">
+          <horizontal_fov>1.22</horizontal_fov>
+          <image>
+            <width>1920</width>
+            <height>1080</height>
+            <format>R8G8B8</format>
+          </image>
+          <clip>
+            <near>0.02</near>
+            <far>300</far>
+          </clip>
+          <noise>
+            <type>gaussian</type>
+            <mean>0.0</mean>
+            <stddev>0.007</stddev>
+          </noise>
+        </camera>
+        <plugin filename="libgazebo_ros_camera.so" name="HMI_camera_controller">
+          <robotNamespace/>
+          <alwaysOn>true</alwaysOn>
+          <updateRate>0.0</updateRate>
+          <cameraName>HMI_camera</cameraName>
+          <imageTopicName>HMI_image_raw</imageTopicName>
+          <cameraInfoTopicName>HMI_camera_info</cameraInfoTopicName>
+          <frameName>HMI_camera</frameName>
+          <hackBaseline>0.07</hackBaseline>
+        </plugin>
+      </sensor>
+    </gazebo>
+  </xacro:unless>
 </robot>
