Commit message: Upload: Robotiq Hand-E gripper (+ adapt code for both grippers).

File: ur3cranfield_gazebo/urdf/ur3.urdf.xacro (robot description, xacro)
@@ -70,4 +70,8 @@
   <xacro:arg name="tf_prefix" default=""/>
   <xacro:property name="tf_prefix" value="$(arg tf_prefix)"/>
+  <xacro:arg name="robotiq_2f85" default="false"/>
+  <xacro:property name="robotiq_2f85" value="$(arg robotiq_2f85)"/>
+  <xacro:arg name="robotiq_hande" default="false"/>
+  <xacro:property name="robotiq_hande" value="$(arg robotiq_hande)"/>
   <!-- Include XACRO-MACRO file of the UR3: -->
   <xacro:include filename="$(find ur3cranfield_gazebo)/urdf/ur3_macro.urdf.xacro"/>
@@ -79,5 +83,6 @@
     output_recipe_filename="${output_recipe_filename}"
     tf_prefix="${tf_prefix}"
-    />
+    robotiq_2f85="${robotiq_2f85}"
+    robotiq_hande="${robotiq_hande}"/>
   <!-- World link -->
   <link name="world"/>
@@ -109,5 +114,5 @@
     <parent link="${tf_prefix}ur3_stand" />
     <child link = "${tf_prefix}base_link" />
-    <origin xyz="0.0 0.0 0.85" rpy="0.0 0.0 ${pi}" />
+    <origin xyz="0.0 0.0 0.85" rpy="0.0 0.0 0.0" />
   </joint>
   <!-- ARUCO TAGS -->

File: ur3cranfield_gazebo/urdf/ur3_macro.urdf.xacro (robot description, xacro)
@@ -60,5 +60,5 @@
   <xacro:include filename="$(find ur3cranfield_gazebo)/urdf/ur3_common.xacro" />
   <!-- XACRO-MACRO of UR3: -->
-  <xacro:macro name="ur3" params="bringup robot_ip script_filename input_recipe_filename output_recipe_filename tf_prefix">
+  <xacro:macro name="ur3" params="bringup robot_ip robotiq_2f85 robotiq_hande script_filename input_recipe_filename output_recipe_filename tf_prefix">
     <!-- LOAD UR3-Common: -->
     <xacro:ur3_common/>
@@ -66,5 +66,5 @@
     <xacro:unless value="${bringup}">
       <xacro:include filename="$(find ur3cranfield_gazebo)/urdf/ur3_transmission.xacro" />
-      <xacro:ur3_transmission />
+      <xacro:ur3_transmission/>
     </xacro:unless>
     <!-- UR3 - ROS2_CONTROL: -->
@@ -73,4 +73,6 @@
       bringup="${bringup}"
       robot_ip="${robot_ip}"
+      robotiq_2f85="${robotiq_2f85}"
+      robotiq_hande="${robotiq_hande}"
       script_filename="${script_filename}"
       input_recipe_filename="${input_recipe_filename}"
@@ -371,315 +373,17 @@
     </xacro:if>
     <!-- === ROBOTIQ 2f-85 GRIPPER === -->
-    <!-- NOTE: JOINT LIMITS have been slightly augmentated from 0.0 to +-0.05 to avoid errors in MoveIt!2 execution. -->
-    <!-- Robotiq: coupler -->
-    <link name="robotiq_coupler">
-      <visual>
-        <geometry>
-          <mesh filename="file://$(find ur3cranfield_gazebo)/meshes/robotiq2f85/robotiq_85_coupler.stl" />
-        </geometry>
-      </visual>
-      <collision>
-        <geometry>
-          <mesh filename="file://$(find ur3cranfield_gazebo)/meshes/robotiq2f85/robotiq_85_coupler.stl" />
-        </geometry>
-      </collision>
-      <inertial>
-        <origin xyz="2.073e-05   1.45286e-03  -1.1049e-03" rpy="0 0 0" />
-        <mass value="0.168" />
-        <inertia ixx="6.69695624e-05" ixy="5.21511788e-09" ixz="-2.74383009e-08"
-                iyy="7.85088161e-05" iyz="5.41105193e-07" izz="1.41819717e-04"/>
-      </inertial>
-    </link>
-    <joint name="robotiq_coupler_joint" type="fixed">
-      <origin xyz="0 0 0.004" rpy="0 0 ${-pi/2.0}" />
-      <parent link="tool0"/>
-      <child link="robotiq_coupler"/>
-    </joint>
-    <gazebo reference="robotiq_coupler">
-      <mu1>0.9</mu1>
-      <mu2>0.9</mu2>
-      <material>Gazebo/FlatBlack</material>
-    </gazebo>
-    <!-- Robotiq: base_link -->
-    <link name="robotiq_85_base_link">
-      <visual>
-        <geometry>
-          <mesh filename="file://$(find ur3cranfield_gazebo)/meshes/robotiq2f85/visual/robotiq_85_base_link.dae"/>
-        </geometry>
-      </visual>
-      <collision>
-        <geometry>
-          <mesh filename="file://$(find ur3cranfield_gazebo)/meshes/robotiq2f85/collision/robotiq_85_base_link.stl"/>
-        </geometry>
-      </collision>
-      <inertial>
-        <mass value="0.636951" />
-        <origin xyz="0.0 0.0 0.0" />
-        <inertia ixx = "0.000380" ixy = "0.000000" ixz = "0.000000"
-            iyx = "0.000000" iyy = "0.001110" iyz = "0.000000"
-            izx = "0.000000" izy = "0.000000" izz = "0.001171" />
-      </inertial>
-    </link>
-    <joint name="robotiq_85_base_joint" type="fixed">
-      <origin xyz="0 0 0.004" rpy="0 ${-pi/2} ${pi}"/>
-      <parent link="robotiq_coupler"/>
-      <child link="robotiq_85_base_link"/>
-    </joint>
-    <!-- Robotiq: left_knuckle -->
-    <link name="robotiq_85_left_knuckle_link">
-      <visual>
-        <geometry>
-          <mesh filename="file://$(find ur3cranfield_gazebo)/meshes/robotiq2f85/visual/robotiq_85_knuckle_link.dae"/>
-        </geometry>
-      </visual>
-      <collision>
-        <geometry>
-          <mesh filename="file://$(find ur3cranfield_gazebo)/meshes/robotiq2f85/collision/robotiq_85_knuckle_link.stl"/>
-        </geometry>
-      </collision>
-      <inertial>
-        <mass value="0.018491" />
-        <origin xyz="0.0 0.0 0.0" />
-        <inertia ixx = "0.000009" ixy = "-0.000001" ixz = "0.000000"
-            iyx = "-0.000001" iyy = "0.000001" iyz = "0.000000"
-            izx = "0.000000" izy = "0.000000" izz = "0.000010" />
-      </inertial>
-    </link>
-    <joint name="robotiq_85_left_knuckle_joint" type="revolute">
-      <parent link="robotiq_85_base_link"/>
-      <child link="robotiq_85_left_knuckle_link"/>
-      <axis xyz="0 0 1"/>
-      <origin rpy="${pi} 0.0 0.0" xyz="0.05490451627 0.03060114443 0.0"/>
-      <limit lower="-0.05" upper="0.80285" velocity="0.5" effort="1000"/>
-      <dynamics damping="1.0" friction="1.0"/>
-    </joint>
-    <!-- Robotiq: right_knuckle -->
-    <link name="robotiq_85_right_knuckle_link">
-      <visual>
-        <geometry>
-          <mesh filename="file://$(find ur3cranfield_gazebo)/meshes/robotiq2f85/visual/robotiq_85_knuckle_link.dae"/>
-        </geometry>
-      </visual>
-      <collision>
-        <geometry>
-          <mesh filename="file://$(find ur3cranfield_gazebo)/meshes/robotiq2f85/collision/robotiq_85_knuckle_link.stl"/>
-        </geometry>
-      </collision>
-      <inertial>
-        <mass value="0.018491" />
-        <origin xyz="0.0 0.0 0.0" />
-        <inertia ixx = "0.000009" ixy = "-0.000001" ixz = "0.000000"
-            iyx = "-0.000001" iyy = "0.000001" iyz = "0.000000"
-            izx = "0.000000" izy = "0.000000" izz = "0.000010" />
-      </inertial>
-    </link>
-    <joint name="robotiq_85_right_knuckle_joint" type="continuous">
-      <parent link="robotiq_85_base_link"/>
-      <child link="robotiq_85_right_knuckle_link"/>
-      <axis xyz="0 0 1"/>
-      <origin rpy="0.0 0.0 0.0" xyz="0.05490451627 -0.03060114443 0.0"/>
-      <limit lower="-0.05" upper="0.80285" velocity="0.5" effort="1000"/>
-      <dynamics damping="1.0" friction="1.0"/>
-    </joint>
-    <!-- Robotiq: left_finger -->
-    <link name="robotiq_85_left_finger_link">
-      <visual>
-        <geometry>
-          <mesh filename="file://$(find ur3cranfield_gazebo)/meshes/robotiq2f85/visual/robotiq_85_finger_link.dae"/>
-        </geometry>
-      </visual>
-      <collision>
-        <geometry>
-          <mesh filename="file://$(find ur3cranfield_gazebo)/meshes/robotiq2f85/collision/robotiq_85_finger_link.stl"/>
-        </geometry>
-      </collision>
-      <inertial>
-        <mass value="0.027309" />
-        <origin xyz="0.0 0.0 0.0" />
-        <inertia ixx = "0.000003" ixy = "-0.000002" ixz = "0.000000"
-            iyx = "-0.000002" iyy = "0.000021" iyz = "0.000000"
-            izx = "0.000000" izy = "0.000000" izz = "0.000020" />
-      </inertial>
-    </link>
-    <joint name="robotiq_85_left_finger_joint" type="fixed">
-      <parent link="robotiq_85_left_knuckle_link"/>
-      <child link="robotiq_85_left_finger_link"/>
-      <origin xyz="-0.00408552455 -0.03148604435 0.0" rpy="0 0 0" />
-      <dynamics damping="1.0" friction="1.0"/>
-    </joint>
-    <!-- Robotiq: right_finger -->
-    <link name="robotiq_85_right_finger_link">
-      <visual>
-        <geometry>
-          <mesh filename="file://$(find ur3cranfield_gazebo)/meshes/robotiq2f85/visual/robotiq_85_finger_link.dae"/>
-        </geometry>
-      </visual>
-      <collision>
-        <geometry>
-          <mesh filename="file://$(find ur3cranfield_gazebo)/meshes/robotiq2f85/collision/robotiq_85_finger_link.stl"/>
-        </geometry>
-      </collision>
-      <inertial>
-        <mass value="0.027309" />
-        <origin xyz="0.0 0.0 0.0" />
-        <inertia ixx = "0.000003" ixy = "-0.000002" ixz = "0.000000"
-            iyx = "-0.000002" iyy = "0.000021" iyz = "0.000000"
-            izx = "0.000000" izy = "0.000000" izz = "0.000020" />
-      </inertial>
-    </link>
-    <joint name="robotiq_85_right_finger_joint" type="fixed">
-      <parent link="robotiq_85_right_knuckle_link"/>
-      <child link="robotiq_85_right_finger_link"/>
-      <origin xyz="-0.00408552455 -0.03148604435 0.0" rpy="0 0 0" />
-      <dynamics damping="1.0" friction="1.0"/>
-    </joint>
-    <!-- Robotiq: left_inner_knuckle -->
-    <link name="robotiq_85_left_inner_knuckle_link">
-      <visual>
-        <geometry>
-          <mesh filename="file://$(find ur3cranfield_gazebo)/meshes/robotiq2f85/visual/robotiq_85_inner_knuckle_link.dae"/>
-        </geometry>
-      </visual>
-      <collision>
-        <geometry>
-          <mesh filename="file://$(find ur3cranfield_gazebo)/meshes/robotiq2f85/collision/robotiq_85_inner_knuckle_link.stl"/>
-        </geometry>
-      </collision>
-      <inertial>
-        <mass value="0.029951" />
-        <origin xyz="0.0 0.0 0.0" />
-        <inertia ixx = "0.000039" ixy = "0.000000" ixz = "0.000000"
-            iyx = "0.000000" iyy = "0.000005" iyz = "0.000000"
-            izx = "0.000000" izy = "0.000000" izz = "0.000035" />
-      </inertial>
-    </link>
-    <joint name="robotiq_85_left_inner_knuckle_joint" type="continuous">
-      <parent link="robotiq_85_base_link"/>
-      <child link="robotiq_85_left_inner_knuckle_link"/>
-      <axis xyz="0 0 1"/>
-      <origin xyz="0.06142 0.0127 0" rpy="${pi} 0.0 0.0" />
-      <limit lower="-0.05" upper="0.80285" velocity="0.5" effort="1000"/>
-      <dynamics damping="1.0" friction="1.0"/>
-    </joint>
-    <!-- Robotiq: right_inner_knuckle -->
-    <link name="robotiq_85_right_inner_knuckle_link">
-      <visual>
-        <geometry>
-          <mesh filename="file://$(find ur3cranfield_gazebo)/meshes/robotiq2f85/visual/robotiq_85_inner_knuckle_link.dae"/>
-        </geometry>
-      </visual>
-      <collision>
-        <geometry>
-          <mesh filename="file://$(find ur3cranfield_gazebo)/meshes/robotiq2f85/collision/robotiq_85_inner_knuckle_link.stl"/>
-        </geometry>
-      </collision>
-      <inertial>
-        <mass value="0.029951" />
-        <origin xyz="0.0 0.0 0.0" />
-        <inertia ixx = "0.000039" ixy = "0.000000" ixz = "0.000000"
-            iyx = "0.000000" iyy = "0.000005" iyz = "0.000000"
-            izx = "0.000000" izy = "0.000000" izz = "0.000035" />
-      </inertial>
-    </link>
-    <joint name="robotiq_85_right_inner_knuckle_joint" type="continuous">
-      <parent link="robotiq_85_base_link"/>
-      <child link="robotiq_85_right_inner_knuckle_link"/>
-      <axis xyz="0 0 1"/>
-      <origin xyz="0.06142 -0.0127 0" rpy="0 0 0"/>
-      <limit lower="-0.05" upper="0.80285" velocity="0.5" effort="1000"/>
-      <dynamics damping="1.0" friction="1.0"/>
-    </joint>
-    <!-- Robotiq: left_finger_tip -->
-    <link name="robotiq_85_left_finger_tip_link">
-      <visual>
-        <geometry>
-          <mesh filename="file://$(find ur3cranfield_gazebo)/meshes/robotiq2f85/visual/robotiq_85_finger_tip_link.dae"/>
-        </geometry>
-      </visual>
-      <collision>
-        <geometry>
-          <mesh filename="file://$(find ur3cranfield_gazebo)/meshes/robotiq2f85/collision/robotiq_85_finger_tip_link.stl"/>
-        </geometry>
-      </collision>
-      <inertial>
-        <mass value="0.019555" />
-        <origin xyz="0.0 0.0 0.0" />
-        <inertia ixx = "0.000002" ixy = "0.000000" ixz = "0.000000"
-            iyx = "0.000000" iyy = "0.000005" iyz = "0.000000"
-            izx = "0.000000" izy = "0.000000" izz = "0.000006" />
-      </inertial>
-    </link>
-    <joint name="robotiq_85_left_finger_tip_joint" type="continuous">
-      <parent link="robotiq_85_left_inner_knuckle_link"/>
-      <child link="robotiq_85_left_finger_tip_link"/>
-      <axis xyz="0 0 1"/>
-      <origin xyz="0.04303959807 -0.03759940821 0.0" rpy="0.0 0.0 0.0"/>
-      <limit lower="-0.80285" upper="0.05" velocity="0.5" effort="1000"/>
-      <dynamics damping="1.0" friction="1.0"/>
-    </joint>
-    <!-- Robotiq: right_finger_tip -->
-    <link name="robotiq_85_right_finger_tip_link">
-      <visual>
-        <geometry>
-          <mesh filename="file://$(find ur3cranfield_gazebo)/meshes/robotiq2f85/visual/robotiq_85_finger_tip_link.dae"/>
-        </geometry>
-      </visual>
-      <collision>
-        <geometry>
-          <mesh filename="file://$(find ur3cranfield_gazebo)/meshes/robotiq2f85/collision/robotiq_85_finger_tip_link.stl"/>
-        </geometry>
-      </collision>
-      <inertial>
-        <mass value="0.019555" />
-        <origin xyz="0.0 0.0 0.0" />
-        <inertia ixx = "0.000002" ixy = "0.000000" ixz = "0.000000"
-            iyx = "0.000000" iyy = "0.000005" iyz = "0.000000"
-            izx = "0.000000" izy = "0.000000" izz = "0.000006" />
-      </inertial>
-    </link>
-    <joint name="robotiq_85_right_finger_tip_joint" type="continuous">
-      <parent link="robotiq_85_right_inner_knuckle_link"/>
-      <child link="robotiq_85_right_finger_tip_link"/>
-      <axis xyz="0 0 1"/>
-      <origin rpy="0.0 0.0 0.0" xyz="0.04303959807 -0.03759940821  0.0"/>
-      <limit lower="-0.80285" upper="0.05" velocity="0.5" effort="1000"/>
-      <dynamics damping="1.0" friction="1.0"/>
-    </joint>
-    <!-- SMALL CUBE FOR GRIPPER PLUGIN -->
-    <link name="EE_robotiq_2f85">
-      <inertial>
-        <origin xyz="0 0 0" rpy="0 0 0" />
-        <mass value="0.00001" />
-        <inertia ixx="0.001" ixy="0.0" ixz="0.0" iyy="0.001" iyz="0.0" izz="0.001"/>
-      </inertial>
-      <visual>
-        <geometry>
-          <box size= "0.001 0.001 0.001" />
-        </geometry>
-      </visual>
-    </link>
-    <xacro:unless value="${bringup}">
-      <joint name="EE_robotiq_2f85_joint" type="prismatic" >
-        <parent link="robotiq_85_base_link" />
-        <child link="EE_robotiq_2f85" />
-        <limit effort="10000" lower="0.0" upper="0.0" velocity="0.0"/>
-        <axis xyz="1 0 0" />
-        <origin xyz="0.128 0.0 0.0" rpy="0 0 0"/>
-      </joint>
-      <!-- LOAD LinkPose Gazebo (ROS2) PLUGIN: -->
-      <gazebo>
-        <plugin name="ros2_linkpose_plugin" filename="libros2_linkpose_plugin.so" >
-          <link>EE_robotiq_2f85</link>
-        </plugin>
-      </gazebo>
-    </xacro:unless>
-    <xacro:if value="${bringup}">
-      <joint name="EE_robotiq_2f85_joint" type="fixed" >
-        <parent link="robotiq_85_base_link" />
-        <child link="EE_robotiq_2f85" />
-        <origin xyz="0.128 0.0 0.0" rpy="0 0 0"/>
-      </joint>
+    <xacro:if value="${robotiq_2f85}">
+      <xacro:include filename="$(find ur3cranfield_gazebo)/urdf/robotiq_2f85.urdf.xacro"/>
+      <xacro:robotiq_2f85
+        bringup="${bringup}"
+      />
     </xacro:if>
-    <!-- === ROBOTIQ 2f-85 GRIPPER === -->
+    <!-- === ROBOTIQ HAND-E GRIPPER === -->
+    <xacro:if value="${robotiq_hande}">
+      <xacro:include filename="$(find ur3cranfield_gazebo)/urdf/robotiq_hande.urdf.xacro"/>
+      <xacro:robotiq_hande
+        bringup="${bringup}"
+      />
+    </xacro:if>
   </xacro:macro>
 </robot>
