Commit message: Upload: Robotiq Hand-E gripper (+ adapt code for both grippers).

File: ur3cranfield_gazebo/urdf/ur3_ros2control.xacro (robot description, xacro)
@@ -99,5 +99,5 @@
   <xacro:property name="keep_alive_count" value="$(arg keep_alive_count)"/>
   <!-- UR3_CONTROL: -->
-  <xacro:macro name="ur3_ros2control" params="bringup robot_ip script_filename input_recipe_filename output_recipe_filename tf_prefix" >
+  <xacro:macro name="ur3_ros2control" params="bringup robotiq_2f85 robotiq_hande robot_ip script_filename input_recipe_filename output_recipe_filename tf_prefix" >
     <!-- 1. ROS2_CONTROL tag name: -->
     <!-- A. GAZEBO SIMULATION: -->
@@ -111,9 +111,8 @@
     <!-- 2. IF GAZEBO -> Load PLUGIN: -->
     <xacro:unless value="${bringup}">
-      <!-- ========== Robotiq 2f-85 ========== -->
       <gazebo>
-        <plugin filename="libgazebo_ros2_control.so" name="gazebo_ros2_control">
+        <plugin filename="libgazebo_ros2_control.so" name="gazebo_ros2_control_ur3">
           <robot_sim_type>gazebo_ros2_control/GazeboSystem</robot_sim_type>
-          <parameters>$(find ur3cranfield_gazebo)/config/urrobotiq_controller.yaml</parameters>
+          <parameters>$(find ur3cranfield_gazebo)/config/ur_controller.yaml</parameters>
         </plugin>
       </gazebo>
@@ -160,5 +159,5 @@
           <state_interface name="force.x"/>
           <state_interface name="force.y"/>
-          <state_interface name="force.z"/> False
+          <state_interface name="force.z"/>
           <state_interface name="torque.x"/>
           <state_interface name="torque.y"/>
@@ -271,5 +270,5 @@
         </command_interface>
         <state_interface name="position">
-          <param name="initial_value">0.0</param>
+          <param name="initial_value">${-pi/2}</param>
         </state_interface>
         <state_interface name="velocity">
@@ -281,96 +280,4 @@
       </joint>
       <xacro:unless value="${bringup}">
-      <!-- === ROBOTIQ 2f-85 GRIPPER === -->
-        <joint name="robotiq_85_left_knuckle_joint">
-          <command_interface name="position">
-            <param name="min">-0.05</param>
-            <param name="max">0.80285</param>
-          </command_interface>
-          <command_interface name="velocity">
-            <param name="min">0.5</param>
-            <param name="max">0.5</param>
-          </command_interface>
-          <state_interface name="position">
-            <param name="initial_value">0.0</param>
-          </state_interface>
-          <state_interface name="velocity"/>
-          <state_interface name="effort"/>
-        </joint>
-        <joint name="robotiq_85_right_knuckle_joint">
-          <command_interface name="position">
-            <param name="min">-0.05</param>
-            <param name="max">0.80285</param>
-          </command_interface>
-          <command_interface name="velocity">
-            <param name="min">0.5</param>
-            <param name="max">0.5</param>
-          </command_interface>
-          <state_interface name="position">
-            <param name="initial_value">0.0</param>
-          </state_interface>
-          <state_interface name="velocity"/>
-          <state_interface name="effort"/>
-        </joint>
-        <joint name="robotiq_85_left_inner_knuckle_joint">
-          <command_interface name="position">
-            <param name="min">-0.05</param>
-            <param name="max">0.80285</param>
-          </command_interface>
-          <command_interface name="velocity">
-            <param name="min">0.5</param>
-            <param name="max">0.5</param>
-          </command_interface>
-          <state_interface name="position">
-            <param name="initial_value">0.0</param>
-          </state_interface>
-          <state_interface name="velocity"/>
-          <state_interface name="effort"/>
-        </joint>
-        <joint name="robotiq_85_right_inner_knuckle_joint">
-          <command_interface name="position">
-            <param name="min">-0.05</param>
-            <param name="max">0.80285</param>
-          </command_interface>
-          <command_interface name="velocity">
-            <param name="min">0.5</param>
-            <param name="max">0.5</param>
-          </command_interface>
-          <state_interface name="position">
-            <param name="initial_value">0.0</param>
-          </state_interface>
-          <state_interface name="velocity"/>
-          <state_interface name="effort"/>
-        </joint>
-        <joint name="robotiq_85_left_finger_tip_joint">
-          <command_interface name="position">
-            <param name="min">-0.80285</param>
-            <param name="max">0.05</param>
-          </command_interface>
-          <command_interface name="velocity">
-            <param name="min">0.5</param>
-            <param name="max">0.5</param>
-          </command_interface>
-          <state_interface name="position">
-            <param name="initial_value">0.0</param>
-          </state_interface>
-          <state_interface name="velocity"/>
-          <state_interface name="effort"/>
-        </joint>
-        <joint name="robotiq_85_right_finger_tip_joint">
-          <command_interface name="position">
-            <param name="min">-0.80285</param>
-            <param name="max">0.05</param>
-          </command_interface>
-          <command_interface name="velocity">
-            <param name="min">0.5</param>
-            <param name="max">0.5</param>
-          </command_interface>
-          <state_interface name="position">
-            <param name="initial_value">0.0</param>
-          </state_interface>
-          <state_interface name="velocity"/>
-          <state_interface name="effort"/>
-        </joint>
-      <!-- === ROBOTIQ 2f-85 GRIPPER === -->
         <joint name="BASE_TF_joint">
           <command_interface name="position"/>
@@ -385,12 +292,16 @@
           <state_interface name="velocity"/>
         </joint>
-        <joint name="EE_robotiq_2f85_joint">
-          <command_interface name="position"/>
-          <command_interface name="velocity"/>
-          <state_interface name="position"/>
-          <state_interface name="velocity"/>
-        </joint>
+        <!-- END EFFECTORS -->
+        <xacro:if value="${robotiq_2f85}">
+          <xacro:include filename="$(find ur3cranfield_gazebo)/urdf/robotiq_2f85.urdf.xacro" />
+          <xacro:robotiq_2f85_ros2control/>
+        </xacro:if>
+        <xacro:if value="${robotiq_hande}">
+          <xacro:include filename="$(find ur3cranfield_gazebo)/urdf/robotiq_hande.urdf.xacro" />
+          <xacro:robotiq_hande_ros2control/>
+        </xacro:if>
       </xacro:unless>
     </ros2_control>
+    <!-- EXTRA: Disable Gazebo collisions -->
     <xacro:unless value="${bringup}">
       <gazebo reference="shoulder_link">
@@ -412,33 +323,4 @@
         <selfCollide>false</selfCollide>
       </gazebo>
-      <!-- === ROBOTIQ 2f-85 GRIPPER === -->
-      <gazebo reference="robotiq_85_base_link">
-        <selfCollide>false</selfCollide>
-      </gazebo>
-      <gazebo reference="robotiq_85_left_knuckle_link">
-        <selfCollide>false</selfCollide>
-      </gazebo>
-      <gazebo reference="robotiq_85_right_knuckle_link">
-        <selfCollide>false</selfCollide>
-      </gazebo>
-      <gazebo reference="robotiq_85_left_finger_link">
-        <selfCollide>false</selfCollide>
-      </gazebo>
-      <gazebo reference="robotiq_85_right_finger_link">
-        <selfCollide>false</selfCollide>
-      </gazebo>
-      <gazebo reference="robotiq_85_left_inner_knuckle_link">
-        <selfCollide>false</selfCollide>
-      </gazebo>
-      <gazebo reference="robotiq_85_right_inner_knuckle_link">
-        <selfCollide>false</selfCollide>
-      </gazebo>
-      <gazebo reference="robotiq_85_left_finger_tip_link">
-        <selfCollide>false</selfCollide>
-      </gazebo>
-      <gazebo reference="robotiq_85_right_finger_tip_link">
-        <selfCollide>false</selfCollide>
-      </gazebo>
-    <!-- ========== END-EFFECTORS ========== -->
       <gazebo reference="end_effector_frame_fixed_joint">
         <preserveFixedJoint>true</preserveFixedJoint>

File: ur3cranfield_gazebo/urdf/ur3_transmission.xacro (robot description, xacro)
@@ -112,60 +112,4 @@
       </actuator>
     </transmission>
-    <!-- === ROBOTIQ 2f-85 GRIPPER === -->
-    <transmission name="robotiq_85_left_knuckle_trans">
-      <type>transmission_interface/SimpleTransmission</type>
-      <joint name="robotiq_85_left_knuckle_joint">
-        <hardwareInterface>hardware_interface/PositionJointInterface</hardwareInterface>
-      </joint>
-      <actuator name="robotiq_85_left_knuckle_motor">
-        <mechanicalReduction>1</mechanicalReduction>
-      </actuator>
-    </transmission>
-    <transmission name="robotiq_85_right_knuckle_trans">
-      <type>transmission_interface/SimpleTransmission</type>
-      <joint name="robotiq_85_right_knuckle_joint">
-        <hardwareInterface>hardware_interface/PositionJointInterface</hardwareInterface>
-      </joint>
-      <actuator name="robotiq_85_right_knuckle_motor">
-        <mechanicalReduction>1</mechanicalReduction>
-      </actuator>
-    </transmission>
-    <transmission name="robotiq_85_left_inner_knuckle_trans">
-      <type>transmission_interface/SimpleTransmission</type>
-      <joint name="robotiq_85_left_inner_knuckle_joint">
-        <hardwareInterface>hardware_interface/PositionJointInterface</hardwareInterface>
-      </joint>
-      <actuator name="robotiq_85_left_inner_knuckle_motor">
-        <mechanicalReduction>1</mechanicalReduction>
-      </actuator>
-    </transmission>
-    <transmission name="robotiq_85_right_inner_knuckle_trans">
-      <type>transmission_interface/SimpleTransmission</type>
-      <joint name="robotiq_85_right_inner_knuckle_joint">
-        <hardwareInterface>hardware_interface/PositionJointInterface</hardwareInterface>
-      </joint>
-      <actuator name="robotiq_85_right_inner_knuckle_motor">
-        <mechanicalReduction>1</mechanicalReduction>
-      </actuator>
-    </transmission>
-    <transmission name="robotiq_85_left_finger_tip_trans">
-      <type>transmission_interface/SimpleTransmission</type>
-      <joint name="robotiq_85_left_finger_tip_joint">
-        <hardwareInterface>hardware_interface/PositionJointInterface</hardwareInterface>
-      </joint>
-      <actuator name="robotiq_85_left_finger_tip_motor">
-        <mechanicalReduction>1</mechanicalReduction>
-      </actuator>
-    </transmission>
-    <transmission name="robotiq_85_right_finger_tip_trans">
-      <type>transmission_interface/SimpleTransmission</type>
-      <joint name="robotiq_85_right_finger_tip_joint">
-        <hardwareInterface>hardware_interface/PositionJointInterface</hardwareInterface>
-      </joint>
-      <actuator name="robotiq_85_right_finger_tip_motor">
-        <mechanicalReduction>1</mechanicalReduction>
-      </actuator>
-    </transmission>
-    <!-- === ROBOTIQ 2f-85 GRIPPER === -->
   </xacro:macro>
 </robot>

Commit message: Modify ArUco Markers to improve detection.

File: ur3cranfield_gazebo/urdf/ur3.urdf.xacro (robot description, xacro)
@@ -139,5 +139,5 @@
       <parent link="${tf_prefix}ur3_stand"/>
       <child link="aruco100"/>
-      <origin xyz="-0.26 0.365 0.845" rpy="0.0 0.0 3.1416" />
+      <origin xyz="0.0 0.0 0.0" rpy="0.0 0.0 0.0" />
     </joint>
     <link name="aruco101">
@@ -162,5 +162,5 @@
       <parent link="${tf_prefix}ur3_stand"/>
       <child link="aruco101"/>
-      <origin xyz="0.26 0.365 0.845" rpy="0.0 0.0 1.5708" />
+      <origin xyz="0.0 0.0 0.0" rpy="0.0 0.0 0.0" />
     </joint>
     <link name="aruco102">
@@ -185,5 +185,5 @@
       <parent link="${tf_prefix}ur3_stand"/>
       <child link="aruco102"/>
-      <origin xyz="-0.26 0.115 0.845" rpy="0.0 0.0 -1.5708" />
+      <origin xyz="0.0 0.0 0.0" rpy="0.0 0.0 0.0" />
     </joint>
     <link name="aruco103">
@@ -208,5 +208,5 @@
       <parent link="${tf_prefix}ur3_stand"/>
       <child link="aruco103"/>
-      <origin xyz="0.26 0.115 0.845" rpy="0.0 0.0 0.0" />
+      <origin xyz="0.0 0.0 0.0" rpy="0.0 0.0 0.0" />
     </joint>
   </xacro:unless>

Commit message: Upload: CubeTray for CubePP task.

File: ur3cranfield_gazebo/urdf/ur3.urdf.xacro (robot description, xacro)
@@ -116,4 +116,28 @@
     <origin xyz="0.0 0.0 0.85" rpy="0.0 0.0 0.0" />
   </joint>
+  <!-- CubeTray -->
+  <link name="CubeTray">
+      <visual>
+        <origin xyz="0.0 0.0 0.0" rpy="0 0 0" />
+        <geometry>
+          <mesh filename="file://$(find ur3cranfield_gazebo)/meshes/ur3stand/CubeTray.dae" scale="1 1 1" />
+        </geometry>
+      </visual>
+      <collision>
+        <origin xyz="0.0 0.0 0.0" rpy="0 0 0" />
+        <geometry>
+          <mesh filename="file://$(find ur3cranfield_gazebo)/meshes/ur3stand/CubeTray.dae" scale="1 1 1" />
+        </geometry>
+      </collision>
+      <inertial>
+        <mass value="100.0"/>
+        <inertia ixx="0.0002" ixy="0.0002" ixz="0.0002" iyy="0.0" iyz="0.0" izz="0.0" />
+      </inertial>
+    </link>
+    <joint name="cell-CubeTray-fixed" type="fixed">
+      <parent link="${tf_prefix}ur3_stand"/>
+      <child link="CubeTray"/>
+      <origin xyz="0.0 0.0 0.0" rpy="0.0 0.0 0.0" />
+    </joint>
   <!-- ARUCO TAGS -->
   <xacro:unless value="${bringup}">
