Commit message: Add coupling bracket to UR3-HandE mount, and adapt waypoints.

File: ur3cranfield_gazebo/urdf/robotiq_hande.urdf.xacro (robot description, xacro)
@@ -61,14 +61,14 @@
     <!-- PART 1: LINK+JOINT TREE -->
     <!-- ======================= -->
-    <!-- Robotiq: coupler -->
-    <link name="robotiq_coupler">
-      <visual>
-        <geometry>
-          <mesh filename="file://$(find ur3cranfield_gazebo)/meshes/robotiqhande/robotiq_hande_coupler.stl" />
-        </geometry>
-      </visual>
-      <collision>
-        <geometry>
-          <mesh filename="file://$(find ur3cranfield_gazebo)/meshes/robotiqhande/robotiq_hande_coupler.stl" />
+    <!-- Robotiq: bracket -->
+    <link name="robotiq_bracket">
+      <visual>
+        <geometry>
+          <mesh filename="file://$(find ur3cranfield_gazebo)/meshes/robotiqhande/hande_bracket.dae" />
+        </geometry>
+      </visual>
+      <collision>
+        <geometry>
+          <mesh filename="file://$(find ur3cranfield_gazebo)/meshes/robotiqhande/hande_bracket.dae" />
         </geometry>
       </collision>
@@ -80,7 +80,31 @@
       </inertial>
     </link>
+    <joint name="robotiq_bracket_joint" type="fixed">
+      <origin xyz="0 0 0.002" rpy="0 0 0" />
+      <parent link="tool0"/>
+      <child link="robotiq_bracket"/>
+    </joint>
+    <!-- Robotiq: coupler -->
+    <link name="robotiq_coupler">
+      <visual>
+        <geometry>
+          <mesh filename="file://$(find ur3cranfield_gazebo)/meshes/robotiqhande/robotiq_hande_coupler.stl" />
+        </geometry>
+      </visual>
+      <collision>
+        <geometry>
+          <mesh filename="file://$(find ur3cranfield_gazebo)/meshes/robotiqhande/robotiq_hande_coupler.stl" />
+        </geometry>
+      </collision>
+      <inertial>
+        <origin xyz="2.073e-05   1.45286e-03  -1.1049e-03" rpy="0 0 0" />
+        <mass value="0.25" />
+        <inertia ixx="6.69695624e-05" ixy="5.21511788e-09" ixz="-2.74383009e-08"
+                iyy="7.85088161e-05" iyz="5.41105193e-07" izz="1.41819717e-04"/>
+      </inertial>
+    </link>
     <joint name="robotiq_coupler_joint" type="fixed">
-      <origin xyz="0 0 -0.009" rpy="0 0 ${-pi/2.0}" />
-      <parent link="tool0"/>
+      <origin xyz="0 0 0" rpy="0 0 0" />
+      <parent link="robotiq_bracket"/>
       <child link="robotiq_coupler"/>
     </joint>
@@ -112,5 +136,5 @@
     </gazebo>
     <joint name="robotiq_hande_base_joint" type="fixed">
-      <origin xyz="0 0 -0.003" rpy="0 0.0 0.0"/>
+      <origin xyz="0 0.0 0.0175" rpy="0.0 0.0 ${pi}"/>
       <parent link="robotiq_coupler"/>
       <child link="robotiq_hande_base_link"/>

File: ur3cranfield_gazebo/urdf/ur3_ros2control.xacro (robot description, xacro)
@@ -270,5 +270,5 @@
         </command_interface>
         <state_interface name="position">
-          <param name="initial_value">${-pi/2}</param>
+          <param name="initial_value">0.0</param>
         </state_interface>
         <state_interface name="velocity">
