Commit message: Prepare ur3cranfield packages for HMI demo.

File: ur3cranfield_gazebo/urdf/ur3cranfield_1.urdf.xacro (robot description, xacro)
@@ -38,4 +38,6 @@
   <xacro:arg name="EE_name" default="none"/>
   <xacro:property name="EE_name" value="$(arg EE_name)"/>
+  <xacro:arg name="hmi" default="false"/>
+  <xacro:property name="hmi" value="$(arg hmi)"/>
   <!-- UR3 Control ARGUMENTS -->
   <xacro:arg name="script_filename" default="none"/>
@@ -99,3 +101,15 @@
     <origin xyz="0.0 0.0 0.85" rpy="0.0 0.0 0.0" />
   </joint>
+  <!-- ros2srrc_HMI CAMERA -->
+  <xacro:if value="${hmi}">
+    <xacro:include filename="$(find ros2srrc_hmi)/urdf/hmicamera.urdf.xacro"/>
+    <xacro:HMI_camera
+      x="2.0"
+      y="1.25"
+      z="1.70"
+      roll="0.0"
+      pitch="0.35"
+      yaw="-2.6"
+    />
+  </xacro:if>
 </robot>

File: ur3cranfield_gazebo/urdf/ur3cranfield_2.urdf.xacro (robot description, xacro)
@@ -38,4 +38,6 @@
   <xacro:arg name="EE_name" default="none"/>
   <xacro:property name="EE_name" value="$(arg EE_name)"/>
+  <xacro:arg name="hmi" default="false"/>
+  <xacro:property name="hmi" value="$(arg hmi)"/>
   <!-- UR3 Control ARGUMENTS -->
   <xacro:arg name="script_filename" default="none"/>
@@ -157,3 +159,15 @@
     <origin xyz="-0.47 0.0 0.0" rpy="0.0 0.0 0.0" />
   </joint>
+  <!-- ros2srrc_HMI CAMERA -->
+  <xacro:if value="${hmi}">
+    <xacro:include filename="$(find ros2srrc_hmi)/urdf/hmicamera.urdf.xacro"/>
+    <xacro:HMI_camera
+      x="2.0"
+      y="1.25"
+      z="1.70"
+      roll="0.0"
+      pitch="0.35"
+      yaw="-2.6"
+    />
+  </xacro:if>
 </robot>

Commit message: Update UR3-Cranfield: Adapt to ros2srrc_hmi and add README.md files.

File: ur3cranfield_gazebo/urdf/ur3cranfield_1.urdf.xacro (robot description, xacro)
@@ -38,6 +38,4 @@
   <xacro:arg name="EE_name" default="none"/>
   <xacro:property name="EE_name" value="$(arg EE_name)"/>
-  <xacro:arg name="hmi" default="false"/>
-  <xacro:property name="hmi" value="$(arg hmi)"/>
   <!-- UR3 Control ARGUMENTS -->
   <xacro:arg name="script_filename" default="none"/>
@@ -101,15 +99,3 @@
     <origin xyz="0.0 0.0 0.85" rpy="0.0 0.0 0.0" />
   </joint>
-  <!-- ros2srrc_HMI CAMERA -->
-  <xacro:if value="${hmi}">
-    <xacro:include filename="$(find ros2srrc_hmi)/urdf/hmicamera.urdf.xacro"/>
-    <xacro:HMI_camera
-      x="2.0"
-      y="1.25"
-      z="1.70"
-      roll="0.0"
-      pitch="0.35"
-      yaw="-2.6"
-    />
-  </xacro:if>
 </robot>

File: ur3cranfield_gazebo/urdf/ur3cranfield_2.urdf.xacro (robot description, xacro)
@@ -38,6 +38,4 @@
   <xacro:arg name="EE_name" default="none"/>
   <xacro:property name="EE_name" value="$(arg EE_name)"/>
-  <xacro:arg name="hmi" default="false"/>
-  <xacro:property name="hmi" value="$(arg hmi)"/>
   <!-- UR3 Control ARGUMENTS -->
   <xacro:arg name="script_filename" default="none"/>
@@ -159,15 +157,3 @@
     <origin xyz="-0.47 0.0 0.0" rpy="0.0 0.0 0.0" />
   </joint>
-  <!-- ros2srrc_HMI CAMERA -->
-  <xacro:if value="${hmi}">
-    <xacro:include filename="$(find ros2srrc_hmi)/urdf/hmicamera.urdf.xacro"/>
-    <xacro:HMI_camera
-      x="2.0"
-      y="1.25"
-      z="1.70"
-      roll="0.0"
-      pitch="0.35"
-      yaw="-2.6"
-    />
-  </xacro:if>
 </robot>
