Commit message: Fix naming (irb120pe -> ur3cranfield).

File: ur3cranfield_gazebo/urdf/objects/BlackCube.urdf (robot description, URDF)
Before this commit: robot BlackCube, 1 links, 0 joints
Links:
- link BlackCube: geometry collision mesh filename=file://$(find ur3cranfield_gazebo)/meshes/cube/BlackCube.dae; visual mesh filename=file://$(find ur3cranfield_gazebo)/meshes/cube/BlackCube.dae

File: ur3cranfield_gazebo/urdf/objects/BlueCube.urdf (robot description, URDF)
Before this commit: robot BlueCube, 1 links, 0 joints
Links:
- link BlueCube: geometry collision mesh filename=file://$(find ur3cranfield_gazebo)/meshes/cube/BlueCube.dae; visual mesh filename=file://$(find ur3cranfield_gazebo)/meshes/cube/BlueCube.dae

File: ur3cranfield_gazebo/urdf/objects/Cube.urdf (robot description, URDF)
Before this commit: robot Cube, 1 links, 0 joints
Links:
- link Cube: geometry collision mesh filename=file://$(find ur3cranfield_gazebo)/meshes/cube/Cube.dae; visual mesh filename=file://$(find ur3cranfield_gazebo)/meshes/cube/Cube.dae

File: ur3cranfield_gazebo/urdf/objects/WhiteCube.urdf (robot description, URDF)
Before this commit: robot WhiteCube, 1 links, 0 joints
Links:
- link WhiteCube: geometry collision mesh filename=file://$(find ur3cranfield_gazebo)/meshes/cube/WhiteCube.dae; visual mesh filename=file://$(find ur3cranfield_gazebo)/meshes/cube/WhiteCube.dae
