Commit message: Update ur3cranfield to adapt to new changes in ros2srrc.

File: ur3cranfield/urdf/objects/BlackCube.urdf (robot description, URDF)
Before this commit: robot cube, 1 links, 0 joints
Links:
- link ${name}: geometry collision mesh filename=file://$(find ur3cranfield)/meshes/objects/${name}.dae; visual mesh filename=file://$(find ur3cranfield)/meshes/objects/${name}.dae

File: ur3cranfield/urdf/ur3cranfield_1.urdf.xacro (robot description, xacro)
@@ -74,5 +74,5 @@
       <origin xyz="0.0 0.0 0.0" rpy="0 0 0" />
       <geometry>
-        <mesh filename="file://$(find ur3cranfield_gazebo)/meshes/ur3stand/ur3stand_complete.dae" scale="1 1 1" />
+        <mesh filename="file://$(find ur3cranfield)/meshes/ur3stand/ur3stand_complete.dae" scale="1 1 1" />
       </geometry>
     </visual>
@@ -80,5 +80,5 @@
       <origin xyz="0.0 0.0 0.0" rpy="0 0 0" />
       <geometry>
-        <mesh filename="file://$(find ur3cranfield_gazebo)/meshes/ur3stand/ur3stand_complete.dae" scale="1 1 1" />
+        <mesh filename="file://$(find ur3cranfield)/meshes/ur3stand/ur3stand_complete.dae" scale="1 1 1" />
       </geometry>
     </collision>

File: ur3cranfield/urdf/ur3cranfield_2.urdf.xacro (robot description, xacro)
@@ -82,5 +82,5 @@
       <origin xyz="0.0 0.0 0.0" rpy="0 0 0" />
       <geometry>
-        <mesh filename="file://$(find ur3cranfield_gazebo)/meshes/ur3stand/ur3stand_complete.dae" scale="1 1 1" />
+        <mesh filename="file://$(find ur3cranfield)/meshes/ur3stand/ur3stand_complete.dae" scale="1 1 1" />
       </geometry>
     </visual>
@@ -88,5 +88,5 @@
       <origin xyz="0.0 0.0 0.0" rpy="0 0 0" />
       <geometry>
-        <mesh filename="file://$(find ur3cranfield_gazebo)/meshes/ur3stand/ur3stand_complete.dae" scale="1 1 1" />
+        <mesh filename="file://$(find ur3cranfield)/meshes/ur3stand/ur3stand_complete.dae" scale="1 1 1" />
       </geometry>
     </collision>
@@ -113,5 +113,5 @@
       <origin xyz="0.0 0.0 0.0" rpy="0 0 0" />
       <geometry>
-        <mesh filename="file://$(find ur3cranfield_gazebo)/meshes/ur3stand/CubeTray.dae" scale="1 1 1" />
+        <mesh filename="file://$(find ur3cranfield)/meshes/ur3stand/CubeTray.dae" scale="1 1 1" />
       </geometry>
     </visual>
@@ -119,5 +119,5 @@
       <origin xyz="0.0 0.0 0.0" rpy="0 0 0" />
       <geometry>
-        <mesh filename="file://$(find ur3cranfield_gazebo)/meshes/ur3stand/CubeTray.dae" scale="1 1 1" />
+        <mesh filename="file://$(find ur3cranfield)/meshes/ur3stand/CubeTray.dae" scale="1 1 1" />
       </geometry>
     </collision>
@@ -132,5 +132,5 @@
       <origin xyz="0.0 0.0 0.0" rpy="0 0 0" />
       <geometry>
-        <mesh filename="file://$(find ur3cranfield_gazebo)/meshes/ur3stand/CubeTray.dae" scale="1 1 1" />
+        <mesh filename="file://$(find ur3cranfield)/meshes/ur3stand/CubeTray.dae" scale="1 1 1" />
       </geometry>
     </visual>
@@ -138,5 +138,5 @@
       <origin xyz="0.0 0.0 0.0" rpy="0 0 0" />
       <geometry>
-        <mesh filename="file://$(find ur3cranfield_gazebo)/meshes/ur3stand/CubeTray.dae" scale="1 1 1" />
+        <mesh filename="file://$(find ur3cranfield)/meshes/ur3stand/CubeTray.dae" scale="1 1 1" />
       </geometry>
     </collision>

File: ur3cranfield/urdf/ur3cranfield_3.urdf.xacro (robot description, xacro)
@@ -82,5 +82,5 @@
       <origin xyz="0.0 0.0 0.0" rpy="0 0 0" />
       <geometry>
-        <mesh filename="file://$(find ur3cranfield_gazebo)/meshes/ur3stand/ur3stand_complete.dae" scale="1 1 1" />
+        <mesh filename="file://$(find ur3cranfield)/meshes/ur3stand/ur3stand_complete.dae" scale="1 1 1" />
       </geometry>
     </visual>
@@ -88,5 +88,5 @@
       <origin xyz="0.0 0.0 0.0" rpy="0 0 0" />
       <geometry>
-        <mesh filename="file://$(find ur3cranfield_gazebo)/meshes/ur3stand/ur3stand_complete.dae" scale="1 1 1" />
+        <mesh filename="file://$(find ur3cranfield)/meshes/ur3stand/ur3stand_complete.dae" scale="1 1 1" />
       </geometry>
     </collision>
@@ -113,5 +113,5 @@
       <origin xyz="0.0 0.0 0.0" rpy="0 0 0" />
       <geometry>
-        <mesh filename="file://$(find ur3cranfield_gazebo)/meshes/ur3stand/ergobox.dae" scale="1 1 1" />
+        <mesh filename="file://$(find ur3cranfield)/meshes/ur3stand/ergobox.dae" scale="1 1 1" />
       </geometry>
     </visual>
@@ -119,5 +119,5 @@
       <origin xyz="0.0 0.0 0.0" rpy="0 0 0" />
       <geometry>
-        <mesh filename="file://$(find ur3cranfield_gazebo)/meshes/ur3stand/ergobox.dae" scale="1 1 1" />
+        <mesh filename="file://$(find ur3cranfield)/meshes/ur3stand/ergobox.dae" scale="1 1 1" />
       </geometry>
     </collision>
@@ -140,5 +140,5 @@
         <origin xyz="0.0 0.0 0.0" rpy="0 0 0" />
         <geometry>
-          <mesh filename="file://$(find ur3cranfield_gazebo)/meshes/aruco/arucoGrid.dae" scale="1 1 1" />
+          <mesh filename="file://$(find ur3cranfield)/meshes/aruco/arucoGrid.dae" scale="1 1 1" />
         </geometry>
       </visual>
@@ -146,5 +146,5 @@
         <origin xyz="0.0 0.0 0.0" rpy="0 0 0" />
         <geometry>
-          <mesh filename="file://$(find ur3cranfield_gazebo)/meshes/aruco/arucoGrid.dae" scale="1 1 1" />
+          <mesh filename="file://$(find ur3cranfield)/meshes/aruco/arucoGrid.dae" scale="1 1 1" />
         </geometry>
       </collision>
