Commit message: Adapt to GzFortress: Remove LinkAttacher, add camera and adapt urdf files.

File: ur3cranfield/urdf/ur3cranfield_1.urdf.xacro (robot description, xacro)
@@ -60,6 +60,5 @@
   <xacro:unless value="${bringup}">
     <gazebo>
-      <plugin filename="libgazebo_ros2_control.so" name="gazebo_ros2_control">
-        <robot_sim_type>gazebo_ros2_control/GazeboSystem</robot_sim_type>
+      <plugin filename="gz_ros2_control-system" name="gz_ros2_control::GazeboSimROS2ControlPlugin">
         <!-- UR3 Controller -->
         <parameters>$(find ros2srrc_robots)/ur3/config/controller.yaml</parameters>
@@ -85,5 +84,5 @@
     <inertial>
       <mass value="1000.0"/>
-      <inertia ixx="500.0" ixy="500.0" ixz="500.0" iyy="500.0" iyz="500.0" izz="500.0" />
+      <inertia ixx="100.0" ixy="0.0" ixz="0.0" iyy="100.0" iyz="0.0" izz="100.0" />
     </inertial>
   </link>

File: ur3cranfield/urdf/ur3cranfield_2.urdf.xacro (robot description, xacro)
@@ -66,6 +66,5 @@
   <xacro:unless value="${bringup}">
     <gazebo>
-      <plugin filename="libgazebo_ros2_control.so" name="gazebo_ros2_control">
-        <robot_sim_type>gazebo_ros2_control/GazeboSystem</robot_sim_type>
+      <plugin filename="gz_ros2_control-system" name="gz_ros2_control::GazeboSimROS2ControlPlugin">
         <!-- UR3 Controller -->
         <parameters>$(find ros2srrc_robots)/ur3/config/controller.yaml</parameters>
@@ -93,5 +92,5 @@
     <inertial>
       <mass value="1000.0"/>
-      <inertia ixx="500.0" ixy="500.0" ixz="500.0" iyy="500.0" iyz="500.0" izz="500.0" />
+      <inertia ixx="100.0" ixy="0.0" ixz="0.0" iyy="100.0" iyz="0.0" izz="100.0" />
     </inertial>
   </link>
@@ -124,5 +123,5 @@
     <inertial>
       <mass value="10.0"/>
-      <inertia ixx="500.0" ixy="500.0" ixz="500.0" iyy="500.0" iyz="500.0" izz="500.0" />
+      <inertia ixx="100.0" ixy="0.0" ixz="0.0" iyy="100.0" iyz="0.0" izz="100.0" />
     </inertial>
   </link>
@@ -143,5 +142,5 @@
     <inertial>
       <mass value="10.0"/>
-      <inertia ixx="500.0" ixy="500.0" ixz="500.0" iyy="500.0" iyz="500.0" izz="500.0" />
+      <inertia ixx="100.0" ixy="0.0" ixz="0.0" iyy="100.0" iyz="0.0" izz="100.0" />
     </inertial>
   </link>

File: ur3cranfield/urdf/ur3cranfield_3.urdf.xacro (robot description, xacro)
@@ -66,6 +66,5 @@
   <xacro:unless value="${bringup}">
     <gazebo>
-      <plugin filename="libgazebo_ros2_control.so" name="gazebo_ros2_control">
-        <robot_sim_type>gazebo_ros2_control/GazeboSystem</robot_sim_type>
+      <plugin filename="gz_ros2_control-system" name="gz_ros2_control::GazeboSimROS2ControlPlugin">
         <!-- UR3 Controller -->
         <parameters>$(find ros2srrc_robots)/ur3/config/controller.yaml</parameters>
@@ -93,5 +92,5 @@
     <inertial>
       <mass value="1000.0"/>
-      <inertia ixx="500.0" ixy="500.0" ixz="500.0" iyy="500.0" iyz="500.0" izz="500.0" />
+      <inertia ixx="100.0" ixy="0.0" ixz="0.0" iyy="100.0" iyz="0.0" izz="100.0" />
     </inertial>
   </link>
@@ -124,5 +123,5 @@
     <inertial>
       <mass value="10.0"/>
-      <inertia ixx="500.0" ixy="500.0" ixz="500.0" iyy="500.0" iyz="500.0" izz="500.0" />
+      <inertia ixx="100.0" ixy="0.0" ixz="0.0" iyy="100.0" iyz="0.0" izz="100.0" />
     </inertial>
   </link>
@@ -181,15 +180,15 @@
         <mass value="1.0" />
         <origin xyz="0 0 0" rpy="0 0 0"/>
-        <inertia ixx="0.0" ixy="0.0" ixz="0.0" iyy="0.0" iyz="0.0" izz="0.0" />
+        <inertia ixx="0.0005" ixy="0.0" ixz="0.0" iyy="0.0005" iyz="0.0" izz="0.0005"/>
       </inertial>
     </link>
-    <joint name="camera_joint" type="fixed">
-      <origin xyz="0.0 0.32 2.09" rpy="0.0 1.5708 1.5708"/>
-      <parent link="world"/>
-      <child link="camera_link"/>
-    </joint>
     <gazebo reference="camera_link">
       <sensor name="camera" type="camera">
+        <pose>0 0 0 0 0 0</pose>
+        <always_on>true</always_on>
         <update_rate>30</update_rate>
+        <visualize>true</visualize>
+        <!-- Gz Transport topic -->
+        <topic>/camera/image_raw</topic>
         <camera name="head">
           <horizontal_fov>1.22</horizontal_fov>
@@ -199,26 +198,14 @@
             <format>R8G8B8</format>
           </image>
-          <clip>
-            <near>0.02</near>
-            <far>300</far>
-          </clip>
-          <noise>
-            <type>gaussian</type>
-            <mean>0.0</mean>
-            <stddev>0.007</stddev>
-          </noise>
+          <clip><near>0.02</near><far>300</far></clip>
+          <camera_info_topic>/camera/camera_info</camera_info_topic>
         </camera>
-        <plugin filename="libgazebo_ros_camera.so" name="camera_controller">
-          <robotNamespace/>
-          <alwaysOn>true</alwaysOn>
-          <updateRate>0.0</updateRate>
-          <cameraName>camera</cameraName>
-          <imageTopicName>image_raw</imageTopicName>
-          <cameraInfoTopicName>camera_info</cameraInfoTopicName>
-          <frameName>camera</frameName>
-          <hackBaseline>0.07</hackBaseline>
-        </plugin>
       </sensor>
     </gazebo>
+    <joint name="camera_joint" type="fixed">
+      <origin xyz="0.0 0.32 2.09" rpy="0.0 1.5708 1.5708"/>
+      <parent link="world"/>
+      <child link="camera_link"/>
+    </joint>
   </xacro:unless>
 </robot>

Commit message: Add {prefix} to robot urdf files.

File: ur3cranfield/urdf/ur3cranfield_1.urdf.xacro (robot description, xacro)
@@ -39,4 +39,6 @@
   <xacro:arg name="EE_name" default="none"/>
   <xacro:property name="EE_name" value="$(arg EE_name)"/>
+  <xacro:arg name="prefix" default=""/>
+  <xacro:property name="prefix" value="$(arg prefix)"/>
   <!-- UR3 Control ARGUMENTS -->
   <xacro:arg name="script_filename" default="none"/>
@@ -56,4 +58,5 @@
     input_recipe_filename="${input_recipe_filename}"
     output_recipe_filename="${output_recipe_filename}"
+    prefix="${prefix}"
   />
   <!-- Load ROS 2 Gazebo Plugin -->
@@ -70,5 +73,5 @@
   <link name="world"/>
   <!-- Robot Stand: LINK -->
-  <link name='ur3_stand'>
+  <link name='${prefix}ur3_stand'>
     <visual>
       <origin xyz="0.0 0.0 0.0" rpy="0 0 0" />
@@ -89,13 +92,13 @@
   </link>
   <!-- Robot Stand: FIXED JOINT -->
-  <joint name="world_joint" type="fixed">
+  <joint name="${prefix}world_joint" type="fixed">
     <parent link="world" />
-    <child link = "ur3_stand" />
+    <child link = "${prefix}ur3_stand" />
     <origin xyz="0.0 0.0 0.0" rpy="0.0 0.0 0.0" />
   </joint>
   <!-- Robot Stand: Robot+Stand JOINT -->
-  <joint name="ur_joint" type="fixed">
-    <parent link="ur3_stand" />
-    <child link = "base_link" />
+  <joint name="${prefix}ur_joint" type="fixed">
+    <parent link="${prefix}ur3_stand" />
+    <child link = "${prefix}base_link" />
     <origin xyz="0.0 0.0 0.85" rpy="0.0 0.0 0.0" />
   </joint>

File: ur3cranfield/urdf/ur3cranfield_2.urdf.xacro (robot description, xacro)
@@ -39,4 +39,6 @@
   <xacro:arg name="EE_name" default="none"/>
   <xacro:property name="EE_name" value="$(arg EE_name)"/>
+  <xacro:arg name="prefix" default=""/>
+  <xacro:property name="prefix" value="$(arg prefix)"/>
   <!-- UR3 Control ARGUMENTS -->
   <xacro:arg name="script_filename" default="none"/>
@@ -56,4 +58,5 @@
     input_recipe_filename="${input_recipe_filename}"
     output_recipe_filename="${output_recipe_filename}"
+    prefix="${prefix}"
   />
   <!-- Include XACRO-MACRO file of the Robotiq HandE: -->
@@ -61,5 +64,6 @@
   <xacro:robotiq_hande
     bringup="${bringup}"
-    parent_link="tool0"
+    parent_link="${prefix}tool0"
+    prefix="${prefix}"
   />
   <!-- Load ROS 2 Gazebo Plugin -->
@@ -78,5 +82,5 @@
   <link name="world"/>
   <!-- Robot Stand: LINK -->
-  <link name='ur3_stand'>
+  <link name='${prefix}ur3_stand'>
     <visual>
       <origin xyz="0.0 0.0 0.0" rpy="0 0 0" />
@@ -97,17 +101,17 @@
   </link>
   <!-- Robot Stand: FIXED JOINT -->
-  <joint name="world_joint" type="fixed">
+  <joint name="${prefix}world_joint" type="fixed">
     <parent link="world" />
-    <child link = "ur3_stand" />
+    <child link = "${prefix}ur3_stand" />
     <origin xyz="0.0 0.0 0.0" rpy="0.0 0.0 0.0" />
   </joint>
   <!-- Robot Stand: Robot+Stand JOINT -->
-  <joint name="ur_joint" type="fixed">
-    <parent link="ur3_stand" />
-    <child link = "base_link" />
+  <joint name="${prefix}ur_joint" type="fixed">
+    <parent link="${prefix}ur3_stand" />
+    <child link = "${prefix}base_link" />
     <origin xyz="0.0 0.0 0.85" rpy="0.0 0.0 0.0" />
   </joint>
   <!-- CubeTray (1): LINK -->
-  <link name='ur3_CubeTray1'>
+  <link name='${prefix}ur3_CubeTray1'>
     <visual>
       <origin xyz="0.0 0.0 0.0" rpy="0 0 0" />
@@ -128,5 +132,5 @@
   </link>
   <!-- CubeTray (2): LINK -->
-  <link name='ur3_CubeTray2'>
+  <link name='${prefix}ur3_CubeTray2'>
     <visual>
       <origin xyz="0.0 0.0 0.0" rpy="0 0 0" />
@@ -147,13 +151,13 @@
   </link>
   <!-- CubeTray (1) - Joint -->
-  <joint name="CT1_joint" type="fixed">
-    <parent link="ur3_stand" />
-    <child link = "ur3_CubeTray1" />
+  <joint name="${prefix}CT1_joint" type="fixed">
+    <parent link="${prefix}ur3_stand" />
+    <child link = "${prefix}ur3_CubeTray1" />
     <origin xyz="0.0 0.0 0.0" rpy="0.0 0.0 0.0" />
   </joint>
   <!-- CubeTray (2) - Joint -->
-  <joint name="CT2_joint" type="fixed">
-    <parent link="ur3_stand" />
-    <child link = "ur3_CubeTray2" />
+  <joint name="${prefix}CT2_joint" type="fixed">
+    <parent link="${prefix}ur3_stand" />
+    <child link = "${prefix}ur3_CubeTray2" />
     <origin xyz="-0.47 0.0 0.0" rpy="0.0 0.0 0.0" />
   </joint>

File: ur3cranfield/urdf/ur3cranfield_3.urdf.xacro (robot description, xacro)
@@ -39,4 +39,6 @@
   <xacro:arg name="EE_name" default="none"/>
   <xacro:property name="EE_name" value="$(arg EE_name)"/>
+  <xacro:arg name="prefix" default=""/>
+  <xacro:property name="prefix" value="$(arg prefix)"/>
   <!-- UR3 Control ARGUMENTS -->
   <xacro:arg name="script_filename" default="none"/>
@@ -56,4 +58,5 @@
     input_recipe_filename="${input_recipe_filename}"
     output_recipe_filename="${output_recipe_filename}"
+    prefix="${prefix}"
   />
   <!-- Include XACRO-MACRO file of the Robotiq HandE: -->
@@ -61,5 +64,6 @@
   <xacro:robotiq_hande
     bringup="${bringup}"
-    parent_link="tool0"
+    parent_link="${prefix}tool0"
+    prefix="${prefix}"
   />
   <!-- Load ROS 2 Gazebo Plugin -->
@@ -78,5 +82,5 @@
   <link name="world"/>
   <!-- Robot Stand: LINK -->
-  <link name='ur3_stand'>
+  <link name='${prefix}ur3_stand'>
     <visual>
       <origin xyz="0.0 0.0 0.0" rpy="0 0 0" />
@@ -97,17 +101,17 @@
   </link>
   <!-- Robot Stand: FIXED JOINT -->
-  <joint name="world_joint" type="fixed">
+  <joint name="${prefix}world_joint" type="fixed">
     <parent link="world" />
-    <child link = "ur3_stand" />
+    <child link = "${prefix}ur3_stand" />
     <origin xyz="0.0 0.0 0.0" rpy="0.0 0.0 0.0" />
   </joint>
   <!-- Robot Stand: Robot+Stand JOINT -->
-  <joint name="ur_joint" type="fixed">
-    <parent link="ur3_stand" />
-    <child link = "base_link" />
+  <joint name="${prefix}ur_joint" type="fixed">
+    <parent link="${prefix}ur3_stand" />
+    <child link = "${prefix}base_link" />
     <origin xyz="0.0 0.0 0.85" rpy="0.0 0.0 0.0" />
   </joint>
   <!-- ERGOBOX -->
-  <link name="ergobox">
+  <link name="${prefix}ergobox">
     <visual>
       <origin xyz="0.0 0.0 0.0" rpy="0 0 0" />
@@ -128,7 +132,7 @@
   </link>
   <!-- Ergobox: FIXED JOINT -->
-  <joint name="ergobox-ur3stand-fixed" type="fixed">
-    <parent link="ur3_stand"/>
-    <child link="ergobox"/>
+  <joint name="${prefix}ergobox-ur3stand-fixed" type="fixed">
+    <parent link="${prefix}ur3_stand"/>
+    <child link="${prefix}ergobox"/>
     <origin xyz="0.0 0.0 0.0" rpy="0.0 0.0 0.0" />
   </joint>
@@ -136,5 +140,5 @@
   <xacro:unless value="${bringup}">
     <!-- ARUCO GRID -->
-    <link name="aruco_grid">
+    <link name="${prefix}aruco_grid">
       <visual>
         <origin xyz="0.0 0.0 0.0" rpy="0 0 0" />
@@ -154,10 +158,10 @@
       </inertial>
     </link>
-    <joint name="ur3stand-aruco_grid-fixed" type="fixed">
-      <parent link="ur3_stand"/>
-      <child link="aruco_grid"/>
+    <joint name="${prefix}ur3stand-aruco_grid-fixed" type="fixed">
+      <parent link="${prefix}ur3_stand"/>
+      <child link="${prefix}aruco_grid"/>
       <origin xyz="0.0 0.0 0.0" rpy="0.0 0.0 0.0" />
     </joint>
-    <gazebo reference="cell-aruco_grid-fixed">
+    <gazebo reference="${prefix}cell-aruco_grid-fixed">
       <preserveFixedJoint>true</preserveFixedJoint>
     </gazebo>
@@ -165,5 +169,5 @@
   <!-- CAMERA -->
   <xacro:unless value="${bringup}">
-    <link name="camera_link">
+    <link name="${prefix}camera_link">
       <collision>
         <origin xyz="0 0 0" rpy="0 0 0"/>
@@ -184,10 +188,10 @@
       </inertial>
     </link>
-    <joint name="camera_joint" type="fixed">
+    <joint name="${prefix}camera_joint" type="fixed">
       <origin xyz="0.0 0.32 2.09" rpy="0.0 1.5708 1.5708"/>
       <parent link="world"/>
-      <child link="camera_link"/>
+      <child link="${prefix}camera_link"/>
     </joint>
-    <gazebo reference="camera_link">
+    <gazebo reference="${prefix}camera_link">
       <sensor name="camera" type="camera">
         <update_rate>30</update_rate>

Commit message: Add (prefix) to urdf files.

File: ur3cranfield/urdf/ur3cranfield_1.urdf.xacro (robot description, xacro)
@@ -39,4 +39,6 @@
   <xacro:arg name="EE_name" default="none"/>
   <xacro:property name="EE_name" value="$(arg EE_name)"/>
+  <xacro:arg name="prefix" default=""/>
+  <xacro:property name="prefix" value="$(arg prefix)"/>
   <!-- UR3 Control ARGUMENTS -->
   <xacro:arg name="script_filename" default="none"/>
@@ -56,4 +58,5 @@
     input_recipe_filename="${input_recipe_filename}"
     output_recipe_filename="${output_recipe_filename}"
+    prefix="${prefix}"
   />
   <!-- Load ROS 2 Gazebo Plugin -->
@@ -69,5 +72,5 @@
   <link name="world"/>
   <!-- Robot Stand: LINK -->
-  <link name='ur3_stand'>
+  <link name='${prefix}ur3_stand'>
     <visual>
       <origin xyz="0.0 0.0 0.0" rpy="0 0 0" />
@@ -88,13 +91,13 @@
   </link>
   <!-- Robot Stand: FIXED JOINT -->
-  <joint name="world_joint" type="fixed">
+  <joint name="${prefix}world_joint" type="fixed">
     <parent link="world" />
-    <child link = "ur3_stand" />
+    <child link = "${prefix}ur3_stand" />
     <origin xyz="0.0 0.0 0.0" rpy="0.0 0.0 0.0" />
   </joint>
   <!-- Robot Stand: Robot+Stand JOINT -->
-  <joint name="ur_joint" type="fixed">
-    <parent link="ur3_stand" />
-    <child link = "base_link" />
+  <joint name="${prefix}ur_joint" type="fixed">
+    <parent link="${prefix}ur3_stand" />
+    <child link = "${prefix}base_link" />
     <origin xyz="0.0 0.0 0.85" rpy="0.0 0.0 0.0" />
   </joint>

File: ur3cranfield/urdf/ur3cranfield_2.urdf.xacro (robot description, xacro)
@@ -39,4 +39,6 @@
   <xacro:arg name="EE_name" default="none"/>
   <xacro:property name="EE_name" value="$(arg EE_name)"/>
+  <xacro:arg name="prefix" default=""/>
+  <xacro:property name="prefix" value="$(arg prefix)"/>
   <!-- UR3 Control ARGUMENTS -->
   <xacro:arg name="script_filename" default="none"/>
@@ -56,4 +58,5 @@
     input_recipe_filename="${input_recipe_filename}"
     output_recipe_filename="${output_recipe_filename}"
+    prefix="${prefix}"
   />
   <!-- Include XACRO-MACRO file of the Robotiq HandE: -->
@@ -61,5 +64,6 @@
   <xacro:robotiq_hande
     bringup="${bringup}"
-    parent_link="tool0"
+    parent_link="${prefix}tool0"
+    prefix="${prefix}"
   />
   <!-- Load ROS 2 Gazebo Plugin -->
@@ -77,5 +81,5 @@
   <link name="world"/>
   <!-- Robot Stand: LINK -->
-  <link name='ur3_stand'>
+  <link name='${prefix}ur3_stand'>
     <visual>
       <origin xyz="0.0 0.0 0.0" rpy="0 0 0" />
@@ -96,17 +100,17 @@
   </link>
   <!-- Robot Stand: FIXED JOINT -->
-  <joint name="world_joint" type="fixed">
+  <joint name="${prefix}world_joint" type="fixed">
     <parent link="world" />
-    <child link = "ur3_stand" />
+    <child link = "${prefix}ur3_stand" />
     <origin xyz="0.0 0.0 0.0" rpy="0.0 0.0 0.0" />
   </joint>
   <!-- Robot Stand: Robot+Stand JOINT -->
-  <joint name="ur_joint" type="fixed">
-    <parent link="ur3_stand" />
-    <child link = "base_link" />
+  <joint name="${prefix}ur_joint" type="fixed">
+    <parent link="${prefix}ur3_stand" />
+    <child link = "${prefix}base_link" />
     <origin xyz="0.0 0.0 0.85" rpy="0.0 0.0 0.0" />
   </joint>
   <!-- CubeTray (1): LINK -->
-  <link name='ur3_CubeTray1'>
+  <link name='${prefix}ur3_CubeTray1'>
     <visual>
       <origin xyz="0.0 0.0 0.0" rpy="0 0 0" />
@@ -127,5 +131,5 @@
   </link>
   <!-- CubeTray (2): LINK -->
-  <link name='ur3_CubeTray2'>
+  <link name='${prefix}ur3_CubeTray2'>
     <visual>
       <origin xyz="0.0 0.0 0.0" rpy="0 0 0" />
@@ -146,13 +150,13 @@
   </link>
   <!-- CubeTray (1) - Joint -->
-  <joint name="CT1_joint" type="fixed">
-    <parent link="ur3_stand" />
-    <child link = "ur3_CubeTray1" />
+  <joint name="${prefix}CT1_joint" type="fixed">
+    <parent link="${prefix}ur3_stand" />
+    <child link = "${prefix}ur3_CubeTray1" />
     <origin xyz="0.0 0.0 0.0" rpy="0.0 0.0 0.0" />
   </joint>
   <!-- CubeTray (2) - Joint -->
-  <joint name="CT2_joint" type="fixed">
-    <parent link="ur3_stand" />
-    <child link = "ur3_CubeTray2" />
+  <joint name="${prefix}CT2_joint" type="fixed">
+    <parent link="${prefix}ur3_stand" />
+    <child link = "${prefix}ur3_CubeTray2" />
     <origin xyz="-0.47 0.0 0.0" rpy="0.0 0.0 0.0" />
   </joint>

File: ur3cranfield/urdf/ur3cranfield_3.urdf.xacro (robot description, xacro)
@@ -39,4 +39,6 @@
   <xacro:arg name="EE_name" default="none"/>
   <xacro:property name="EE_name" value="$(arg EE_name)"/>
+  <xacro:arg name="prefix" default=""/>
+  <xacro:property name="prefix" value="$(arg prefix)"/>
   <!-- UR3 Control ARGUMENTS -->
   <xacro:arg name="script_filename" default="none"/>
@@ -56,4 +58,5 @@
     input_recipe_filename="${input_recipe_filename}"
     output_recipe_filename="${output_recipe_filename}"
+    prefix="${prefix}"
   />
   <!-- Include XACRO-MACRO file of the Robotiq HandE: -->
@@ -61,5 +64,6 @@
   <xacro:robotiq_hande
     bringup="${bringup}"
-    parent_link="tool0"
+    parent_link="${prefix}tool0"
+    prefix="${prefix}"
   />
   <!-- Load ROS 2 Gazebo Plugin -->
@@ -77,5 +81,5 @@
   <link name="world"/>
   <!-- Robot Stand: LINK -->
-  <link name='ur3_stand'>
+  <link name='${prefix}ur3_stand'>
     <visual>
       <origin xyz="0.0 0.0 0.0" rpy="0 0 0" />
@@ -96,17 +100,17 @@
   </link>
   <!-- Robot Stand: FIXED JOINT -->
-  <joint name="world_joint" type="fixed">
+  <joint name="${prefix}world_joint" type="fixed">
     <parent link="world" />
-    <child link = "ur3_stand" />
+    <child link = "${prefix}ur3_stand" />
     <origin xyz="0.0 0.0 0.0" rpy="0.0 0.0 0.0" />
   </joint>
   <!-- Robot Stand: Robot+Stand JOINT -->
-  <joint name="ur_joint" type="fixed">
-    <parent link="ur3_stand" />
-    <child link = "base_link" />
+  <joint name="${prefix}ur_joint" type="fixed">
+    <parent link="${prefix}ur3_stand" />
+    <child link = "${prefix}base_link" />
     <origin xyz="0.0 0.0 0.85" rpy="0.0 0.0 0.0" />
   </joint>
   <!-- ERGOBOX -->
-  <link name="ergobox">
+  <link name="${prefix}ergobox">
     <visual>
       <origin xyz="0.0 0.0 0.0" rpy="0 0 0" />
@@ -127,7 +131,7 @@
   </link>
   <!-- Ergobox: FIXED JOINT -->
-  <joint name="ergobox-ur3stand-fixed" type="fixed">
-    <parent link="ur3_stand"/>
-    <child link="ergobox"/>
+  <joint name="${prefix}ergobox-ur3stand-fixed" type="fixed">
+    <parent link="${prefix}ur3_stand"/>
+    <child link="${prefix}ergobox"/>
     <origin xyz="0.0 0.0 0.0" rpy="0.0 0.0 0.0" />
   </joint>
@@ -135,5 +139,5 @@
   <xacro:unless value="${bringup}">
     <!-- ARUCO GRID -->
-    <link name="aruco_grid">
+    <link name="${prefix}aruco_grid">
       <visual>
         <origin xyz="0.0 0.0 0.0" rpy="0 0 0" />
@@ -153,10 +157,10 @@
       </inertial>
     </link>
-    <joint name="ur3stand-aruco_grid-fixed" type="fixed">
-      <parent link="ur3_stand"/>
-      <child link="aruco_grid"/>
+    <joint name="${prefix}ur3stand-aruco_grid-fixed" type="fixed">
+      <parent link="${prefix}ur3_stand"/>
+      <child link="${prefix}aruco_grid"/>
       <origin xyz="0.0 0.0 0.0" rpy="0.0 0.0 0.0" />
     </joint>
-    <gazebo reference="cell-aruco_grid-fixed">
+    <gazebo reference="${prefix}ur3stand-aruco_grid-fixed">
       <preserveFixedJoint>true</preserveFixedJoint>
     </gazebo>
@@ -164,5 +168,5 @@
   <!-- CAMERA -->
   <xacro:unless value="${bringup}">
-    <link name="camera_link">
+    <link name="${prefix}camera_link">
       <collision>
         <origin xyz="0 0 0" rpy="0 0 0"/>
@@ -183,6 +187,6 @@
       </inertial>
     </link>
-    <gazebo reference="camera_link">
-      <sensor name="camera" type="camera">
+    <gazebo reference="${prefix}camera_link">
+      <sensor name="${prefix}camera" type="camera">
         <pose>0 0 0 0 0 0</pose>
         <always_on>true</always_on>
