Commit message: Fix GreenCube -> .dae file path & ArUco grid inertia values.

File: ur3cranfield/urdf/ur3cranfield_3.urdf.xacro (robot description, xacro)
@@ -154,5 +154,5 @@
       <inertial>
         <mass value="10.0"/>
-        <inertia ixx="0.0002" ixy="0.0002" ixz="0.0002" iyy="0.0" iyz="0.0" izz="0.0" />
+        <inertia ixx="0.04" ixy="0.0" ixz="0.0" iyy="0.04" iyz="0.0" izz="0.04" />
       </inertial>
     </link>
